File: powerflex.kicad_sch (KiCad schematic)
At the start: 2 parts, among them CN12 DF40C-20DP-0.4V, CN13 DF40C-20DP-0.4V

Commit message: forgot to save
Connections:
- no-connect marks 0 -> 16
Changed lines of the file:
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@@
 	(generator_version "10.0")
 	(paper "A5")
+	(no_connect
+		(at 152.4 53.34)
+	)
+	(no_connect
+		(at 57.15 53.34)
+	)
+	(no_connect
+		(at 149.86 35.56)
+	)
+	(no_connect
+		(at 157.48 35.56)
+	)
+	(no_connect
+		(at 62.23 35.56)
+	)
+	(no_connect
+		(at 149.86 53.34)
+	)
+	(no_connect
+		(at 57.15 35.56)
+	)
+	(no_connect
+		(at 157.48 53.34)
+	)
+	(no_connect
+		(at 59.69 53.34)
+	)
+	(no_connect
+		(at 62.23 53.34)
+	)
+	(no_connect
+		(at 154.94 35.56)
+	)
+	(no_connect
+		(at 64.77 53.34)
+	)
+	(no_connect
+		(at 152.4 35.56)
+	)
+	(no_connect
+		(at 154.94 53.34)
+	)
+	(no_connect
+		(at 59.69 35.56)
+	)
+	(no_connect
+		(at 64.77 35.56)
+	)
 	(global_label "FerriteGND_PWR"
 		(shape input)
