File: ledbar.kicad_sch (KiCad schematic)
At the start: 91 parts, among them CN18 DF40C-10DP-0.4V

Commit message: finished BOM, replaced discontinued parts, added missing footprints, updated schematics and libraries
Parts:
- C166, C167, C168, C169, C170, C171, C172, C173, C174, C175, C176, C177, C178, C179, C180, C181, C182, C183, C184, C185, C186, C187, C188, C189, C190, C191, C192, C193, C194, C195, C196, C197, C198, C199, C200, C201, C202, C203, C204, C205, C206, C207, C208, C209, C210: LCSC Part (none) -> C1591

Commit message: imported footprints and 3d models, replaced obsolete components, finished schematic audit, wired new usb hub and flash chip + more, removed stale nets
Parts:
- added C?: 220 µF, symbol Device:C_Small
Connections:
- net GND: now also C?.2
- net LED_5V: now also C?.1
Changed lines of the file:
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@@
 		)
 	)
+	(global_label "LED_5V"
+		(shape input)
+		(at 162.56 40.64 90)
+		(fields_autoplaced yes)
+		(effects
+			(font
+				(size 1.27 1.27)
+			)
+			(justify left)
+		)
+		(property "Intersheetrefs" "${INTERSHEET_REFS}"
+			(at 162.56 30.942 90)
+			(hide yes)
+			(show_name no)
+			(do_not_autoplace no)
+			(effects
+				(font
+					(size 1.27 1.27)
+				)
+				(justify left)
+			)
+		)
+	)
 	(global_label "GND"
 		(shape input)
@@
 	(global_label "GND"
 		(shape input)
+		(at 162.56 45.72 270)
+		(fields_autoplaced yes)
+		(effects
+			(font
+				(size 1.27 1.27)
+			)
+			(justify right)
+		)
+		(property "Intersheetrefs" "${INTERSHEET_REFS}"
+			(at 162.56 52.5757 90)
+			(hide yes)
+			(show_name no)
+			(do_not_autoplace no)
+			(effects
+				(font
+					(size 1.27 1.27)
+				)
+				(justify right)
+			)
+		)
+	)
+	(global_label "GND"
+		(shape input)
 		(at 269.24 270.51 270)
 		(fields_autoplaced yes)
@@
 					(unit 1)
 				)
+			)
+		)
+	)
+	(symbol
+		(lib_id "Device:C_Small")
+		(at 162.56 43.18 0)
+		(unit 1)
+		(body_style 1)
+		(exclude_from_sim no)
+		(in_bom yes)
+		(on_board yes)
+		(in_pos_files yes)
+		(dnp no)
+		(fields_autoplaced yes)
+		(property "Reference" "C?"
+			(at 165.1 41.9162 0)
+			(show_name no)
+			(do_not_autoplace no)
+			(effects
+				(font
+					(size 1.27 1.27)
+				)
+				(justify left)
+			)
+		)
+		(property "Value" "220 µF"
+			(at 165.1 44.4562 0)
+			(show_name no)
+			(do_not_autoplace no)
+			(effects
+				(font
+					(size 1.27 1.27)
+				)
+				(justify left)
+			)
+		)
+		(property "Footprint" ""
+			(at 162.56 43.18 0)
+			(hide yes)
+			(show_name no)
+			(do_not_autoplace no)
+			(effects
+				(font
+					(size 1.27 1.27)
+				)
+			)
+		)
+		(property "Datasheet" ""
+			(at 162.56 43.18 0)
+			(hide yes)
+			(show_name no)
+			(do_not_autoplace no)
+			(effects
+				(font
+					(size 1.27 1.27)
+				)
+			)
+		)
+		(property "Description" "Unpolarized capacitor, small symbol"
+			(at 162.56 43.18 0)
+			(hide yes)
+			(show_name no)
+			(do_not_autoplace no)
+			(effects
+				(font
+					(size 1.27 1.27)
+				)
+			)
+		)
+		(pin "2"
+		)
+		(pin "1"
+		)
+		(instances
+			(project "slate113"
+				(path "/9144d9eb-e8ae-422f-a98d-7eba2889072a"
+					(reference "C?")
+					(unit 1)
+				)

Commit message: configured 8-layer pcb with micro vias, finished power mezzanine routing, completed io port, started work on slateconnect mezzanine
Parts:
- C235: renamed from C?; footprint (none) -> slate113:CHEMI-F61; DigiKey Part (none) -> 565-3163-1-ND; MPN (none) -> APXF6R3ARA221MF61G; Manufacturer (none) -> Chemi-Con
Changed lines of the file:
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@@
 		(dnp no)
 		(fields_autoplaced yes)
-		(property "Reference" "C?"
+		(property "Reference" "C235"
 			(at 165.1 41.9162 0)
 			(show_name no)
@@
 			)
 		)
-		(property "Footprint" ""
+		(property "Footprint" "slate113:CHEMI-F61"
 			(at 162.56 43.18 0)
 			(hide yes)
@@
 			)
 		)
+		(property "Manufacturer" "Chemi-Con"
+			(at 162.56 43.18 0)
+			(hide yes)
+			(show_name no)
+			(do_not_autoplace no)
+			(effects
+				(font
+					(size 1.27 1.27)
+				)
+			)
+		)
+		(property "MPN" "APXF6R3ARA221MF61G"
+			(at 162.56 43.18 0)
+			(hide yes)
+			(show_name no)
+			(do_not_autoplace no)
+			(effects
+				(font
+					(size 1.27 1.27)
+				)
+			)
+		)
+		(property "DigiKey Part" "565-3163-1-ND"
+			(at 162.56 43.18 0)
+			(hide yes)
+			(show_name no)
+			(do_not_autoplace no)
+			(effects
+				(font
+					(size 1.27 1.27)
+				)
+			)
+		)
 		(pin "2"
 		)
@@
 			(project "slate113"
 				(path "/9144d9eb-e8ae-422f-a98d-7eba2889072a"
-					(reference "C?")
+					(reference "C235")
 					(unit 1)
 				)
