File: radio.kicad_sch (KiCad schematic)
At the start: 87 parts, among them CN20 DF40C-24DP-0.4V, J19 U.FL, J20 U.FL, Q1 NPN, SW3 4*4*1.7, U18 ESP32-S3-WROOM-1U-N8, U19 TXM27.12M0004322DBBDO00T, U20 CC1101RGPR, U21 0896BM15A0001001E, U22 LC29HBA, U23 EM4095HMSO16B+, U24 PE4259-63, U25 PE4259-63, U26 PE4259-63, U27 PE4259-63, U28 0896BM15A0001001E, U29 PN7160A1HN/C100Y, U31 S2B-PH-K-S-GW, U32 S2B-PH-K-S-GW, U33 W25Q128JVSIQTR, U34 SiP32508DT, U35 SiP32508DT, Y1 12MHz, Y3 26.0MHz

Commit message: imported footprints and 3d models, replaced obsolete components, finished schematic audit, wired new usb hub and flash chip + more, removed stale nets
Parts:
- removed C59, C61, C62: 100nF, Capacitor_SMD:C_0603_1608Metric, symbol Device:C_Small
- removed FB4: FerriteBead_Small, symbol Device:FerriteBead_Small
- removed L4: AOTA-B201610S3R3-101-T, slate113:IND-SMD_L2.0-W1.6_AOTA-B201610S3R3-101-T, symbol slate113:AOTA-B201610S3R3-101-T
- removed Q1: NPN, symbol Simulation_SPICE:NPN
- removed R26: 33Ω, Resistor_SMD:R_0603_1608Metric, symbol Device:R_Small
- removed R38: 10kΩ, Resistor_SMD:R_0603_1608Metric, symbol Device:R_Small
- removed SW3: 4*4*1.7, slate113:SW-SMD_4P-L5.2-W5.2-P3.70-LS6.5, symbol slate113:4*4*1.7
- removed U18: ESP32-S3-WROOM-1U-N8, symbol MCU_RaspberryPi:RP2350B
- removed U33: W25Q128JVSIQTR, slate113:SOIC-8_L5.3-W5.3-P1.27-LS8.0-BL, symbol slate113:W25Q128JVSIQTR
- removed Y1: 12MHz, slate113:CRYSTAL-SMD_4P-L3.2-W2.5-BL, symbol Device:Crystal
- added C230: 12 pF ± 5%, symbol Device:C_Small
- added C231: 6.8 pF ± 0.5 pF, symbol Device:C_Small
- added C232: 220 pF ± 5%, symbol Device:C_Small
- added C233, C234: 100nF, symbol Device:C_Small
- added L10, L9: 33 nH ± 5%, Inductor_SMD:L_0402_1005Metric, symbol Device:L
- added Q1: MMBT3904-TP, slate113:SOT-23-3_L2.9-W1.3-P1.90-LS2.4-BR, symbol slate113:MMBT3904-TP
- added R104: 5.1kΩ, Resistor_SMD:R_0603_1608Metric, symbol Device:R_Small
- added R110, R111, R112, R113, R114, R115, R116, R117, R118, R119, R120: 10kΩ, Resistor_SMD:R_0603_1608Metric, symbol Device:R_Small
- added R132, R133: 4.7kΩ, Resistor_SMD:R_0603_1608Metric, symbol Device:R_Small
- added SW3, SW4: SW_Push, symbol Switch:SW_Push
- added U33: ESP32-S3-WROOM-1U-N16R2, slate113:WIRELM-SMD_ESP32-S3-WROOM-1U, symbol slate113:ESP32-S3-WROOM-1U-N8
- added U64: TCA9535PWR, slate113:TSSOP-24_L7.8-W4.4-P0.65-LS6.4-BL, symbol slate113:TCA9535PWR_C130204
- added U71: SKY13373-460LF, slate113:QFN-12_L2.0-W2.0-P0.50-BL-EP, symbol slate113:SKY13373-460LF
- added U72: SN74AXC1T45DCKR, slate113:SC-70-6_L2.0-W1.3-P0.65-LS2.1-BL-1, symbol slate113:SN74AXC1T45DCKR
- C25: value 1µF -> 100nF; LCSC Part C15849 -> C92848; MPN CL10A105KB8NNNC -> UMK107BJ105KA-T; Manufacturer Samsung Electro-Mechanics -> Taiyo Yuden
- C28, C29: value 27pF -> 15pF
- C57: LCSC Part C1591 -> C380317; MPN CL10B104KB8NNNC -> TCC0603X5R106M160CT; Manufacturer (none) -> Samsung Electro-Mechanics
- C58: LCSC Part C1591 -> C380317; MPN CL10B104KB8NNNC -> TCC0603X5R106M160CT
- C65: value 6.8pF -> 6.8 pF ± 0.5 pF; Manufacturer (none) -> Samsung Electro-Mechanics
- C76: LCSC Part C15849 -> C92848; MPN CL10A105KB8NNNC -> UMK107BJ105KA-T; Manufacturer (none) -> Taiyo Yuden
- C82: value 4.7uF -> 100nF; footprint Capacitor_SMD:C_0603_1608Metric -> (none); LCSC Part C19666 -> (none); MPN CL10A475KO8NNNC -> (none); Manufacturer Samsung Electro-Mechanics -> (none)
- C83: value 4.7uF -> 100pF; LCSC Part C19666 -> C14858; MPN CL10A475KO8NNNC -> CL10C101JB8NNNC; Manufacturer Samsung Electro-Mechanics -> (none)
- C84: value 4.7uF -> 100nF; LCSC Part C19666 -> C14858; MPN CL10A475KO8NNNC -> CL10C101JB8NNNC
- C85: value 4.7uF -> 220 pF ± 5%; footprint Capacitor_SMD:C_0603_1608Metric -> (none); LCSC Part C19666 -> (none); MPN CL10A475KO8NNNC -> (none); Manufacturer Samsung Electro-Mechanics -> (none)
- D2: value TVS -> RCLAMP0521PATCT; footprint (none) -> slate113:D0402-BI; DigiKey Part 1727-4154-2-ND -> (none); LCSC Part C19829543 -> C117554; MPN PESD3V3U1UL -> RCLAMP0521PATCT; Manufacturer DigiKey -> Semtech
- D3: value RCLAMP0521PATCT -> PESD3V3U1UL; footprint (none) -> slate113:SOD-882_L1.0-W0.6-RD; DigiKey Part RCLAMP0521PATR-ND -> (none); LCSC Part (none) -> C19829543; MPN RCLAMP0521PATCT -> PESD3V3U1UL; Manufacturer Semtech -> Nexperia
- D4: value TVS -> PESD3V3U1UL; footprint (none) -> slate113:SOD-882_L1.0-W0.6-RD; DigiKey Part 1727-4154-2-ND -> (none); Manufacturer DigiKey -> Nexperia
- FB5: footprint (none) -> Inductor_SMD:L_0603_1608Metric
- L6, L7: value 33nH -> 33 nH ± 5%
- R42: LCSC Part C23162 -> C163914; MPN 0603WAF4701T5E -> WR06X4701FTL; Manufacturer (none) -> Walsin
- R43: LCSC Part C22859 -> C109318; MPN 0603WAF100JT5E -> RC0603FR-0710RL; Manufacturer (none) -> Yageo
- U23: DigiKey Part (none) -> 2651-EM4095HMSO16B+CT-ND; LCSC Part C17203964 -> (none)
- U24, U25, U26, U27: DigiKey Part (none) -> 1046-1011-1-ND
- U28: value 0896BM15A0001001E -> 0433BM15A0001001E; DigiKey Part (none) -> 712-0433BM15A0001001ECT-ND; LCSC Part C2917678 -> (none); MPN 0896BM15A0001001E -> 0433BM15A0001001E; Manufacturer LCSC -> Johanson
- U29: value PN7160A1HN/C100Y -> PN7160A1HN/C100E; DigiKey Part (none) -> 568-PN7160A1HN/C100E-ND; LCSC Part C3303790 -> (none); MPN PN7160A1HN/C100Y -> PN7160A1HN/C100E
Connections:
- net 315MHZ_OUT: now also C232.1, U71.1 (J1); no longer C63.1, C65.2, J19.1 (In), U28.1 (UNBALANCEDPORT)
- net 3V3: now also C58.2, C82.1, C233.1, R104.1, R132.2, R133.1, U33.2 (3V3), U64.24 (VCC), U71.6 (VDD), U72.1 (VCCA), U72.5 (DIR); no longer C57.1, C58.1, U20.11 (AVDD), U20.14 (AVDD), U20.15 (AVDD), U20.9 (AVDD)
- net BADUSB_DM: now also U33.13 (IO19)
- net BADUSB_DP: now also U33.14 (IO20)
- net BAND_SEL_1: now also U64.6 (P02)
- net BAND_SEL_2: now also U64.7 (P03)
- net CC_GDO0: now also U33.6 (IO6)
- net CC_GDO2: now also U33.25 (IO48)
- net CM5_UART_RX: now also U33.11 (IO18)
- net CM5_UART_TX: now also U33.10 (IO17), U72.3 (A)
- net EM_DEMOD_OUT: now also U33.4 (IO4)
- net EM_MOD: now also U33.32 (IO39)
- net EM_RDY_CLK: now also U33.23 (IO21)
- net EM_SHD: now also R112.1, U64.9 (P05)
- net GND: now also C57.1, C58.1, C65.2, C84.1, C230.1, C231.1, C233.2, C234.2, Q1.2 (E), R110.2, R111.2, R112.2, R113.2, R114.2, R115.1, R116.1, R117.1, R118.1, R119.1, R120.1, SW3.1, SW4.1, U33.1 (GND), U33.40 (GND), U33.41 (GND), U64.12 (GND), U64.2 (A1), U64.21 (A0), U64.3 (A2), U71.10 (GND), U71.12 (GND), U71.13 (PAD), U71.2 (GND), U71.7 (GND), U71.8 (GND), U72.2 (GND); no longer C57.2, C58.2, C84.2, CN20.16, CN20.18, L6.2, L7.2
- net GPS_1PPS: now also U33.24 (IO47)
- net GPS_ANT: now also D2.2 (A); no longer D3.2 (A)
- net GPS_EN: now also R111.1, U64.5 (P01)
- net GPS_RESET: now also U64.8 (P04)
- net GPS_RESET_N: now also Q1.3 (C)
- net GPS_UART_RX: now also U33.9 (IO16); no longer U22.21 (RXD1/SPI_MOSI)
- net GPS_UART_TX: now also U33.8 (IO15)
- net GPS_VCC: now also D3.2 (A); no longer D2.2 (A)
- net GPS_WAKEUP: now also U33.5 (IO5)
- net GPS_WI: now also U33.29 (IO36)
- net LED_CLK_3V3: now also U33.35 (IO42)
- net LED_DATA_3V3: now also U33.34 (IO41)
- net LED_PWR_EN: now also R110.1, U64.4 (P00)
- net NFC_IRQ: now also U33.30 (IO37)
- net NFC_VEN: now also R114.1, U64.14 (P11)
- net NPN_B: now also Q1.1 (B)
- net RADIO_I2C0_SCL: now also R133.2, U33.17 (IO9), U64.22 (SCL)
- net RADIO_I2C0_SDA: now also R132.1, U33.12 (IO8), U64.23 (SDA)
- net RADIO_SPI0_CS: now also U33.19 (IO11)
- net RADIO_SPI0_MISO: now also U33.18 (IO10)
- net RADIO_SPI0_MOSI: now also U33.21 (IO13)
- net RADIO_SPI0_SCK: now also U33.20 (IO12)
- net RP_ACC_AUX0: now also U64.11 (P07)
- net RP_ACC_AUX1: now also U64.13 (P10)
- net RP_ACC_CS0_N: now also U33.31 (IO38)
- net RP_ACC_IRQ0: now also U33.36 (RXD0)
- net RP_ACC_MISO: now also U33.28 (IO35)
- net RP_ACC_MOSI: now also U33.38 (IO2)
- net RP_ACC_RESET_N: now also R113.1, U64.10 (P06)
- net RP_ACC_SCK: now also U33.33 (IO40)
- net U24_RF1: no longer C64.1
- net U25_RF1: now also C64.1; no longer C64.2
- net at L8.1, R43.2: now also C83.1, C84.2
- net VDD_EXT: now reaches U22.7 (VDD_EXT)
- net VDD_EXT: now also C234.1, U72.6 (VCCB)
- removed net DVDD: C82.1, C83.1, C84.1, C85.1
- net RP_RST renamed ESP_RST
- net ESP_RST: now also C57.2, R104.2, SW3.2, U33.3 (EN)
- new net: C231.2, C232.2, L10.1
- new net: C64.2, L7.2, L9.1
- new net: C85.1, L6.2
- new net: C230.2, L10.2, L9.2
- new net 433MHZ_OUT: U28.1 (UNBALANCEDPORT), U71.9 (J2)
- new net 868/915MHZ_OUT: C63.1, U71.3 (J3)
- new net BOOT: SW4.2, U33.27 (IO0)
- new net CC1101_CAPS: U20.11 (AVDD), U20.14 (AVDD), U20.15 (AVDD), U20.9 (AVDD)
- new net GPS_UART_RX_F: U22.21 (RXD1/SPI_MOSI), U72.4 (B)
- new net RF_V1: CN20.16, U71.4 (V1)
- new net RF_V2: CN20.18, U71.5 (V2)
- new net R_UNUSED: R115.2, R116.2, R117.2, R118.2, R119.2, R120.2, U64.15 (P12), U64.16 (P13), U64.17 (P14), U64.18 (P15), U64.19 (P16), U64.20 (P17)
- new net U.FL_OUT: J19.1 (In), U71.11 (RFC)
- no-connect marks 38 -> 31
Other:
- note added: "RF Switch/Router"
- note added: "Resistors"
- note removed: "BOOTSEL Button"
- note removed: "Flash Chip | 16MB"
- moved on the sheet: C25, C28, C29, C64, C68, C69, C71, C72, C73, C74, C75, C76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

Commit message: configured 8-layer pcb with micro vias, finished power mezzanine routing, completed io port, started work on slateconnect mezzanine
Parts:
- C230, C231, C232, C233, C234, C82, C85: footprint (none) -> Capacitor_SMD:C_0402_1005Metric
- SW3, SW4: footprint (none) -> slate113:KEY-SMD_KMR2XXGXXX; LCSC Part (none) -> C99271; MPN (none) -> KMR231GLFS; Manufacturer (none) -> C&K
Changed lines of the file:
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@@
 			)
 		)
-		(property "Footprint" ""
+		(property "Footprint" "Capacitor_SMD:C_0402_1005Metric"
 			(at 304.8 30.48 0)
 			(hide yes)
@@
 			)
 		)
-		(property "Footprint" ""
+		(property "Footprint" "Capacitor_SMD:C_0402_1005Metric"
 			(at 284.48 41.91 0)
 			(hide yes)
@@
 			)
 		)
-		(property "Footprint" ""
+		(property "Footprint" "Capacitor_SMD:C_0402_1005Metric"
 			(at 361.95 209.55 0)
 			(hide yes)
@@
 			)
 		)
-		(property "Footprint" ""
+		(property "Footprint" "Capacitor_SMD:C_0402_1005Metric"
 			(at 389.89 209.55 0)
 			(hide yes)
@@
 			)
 		)
-		(property "Footprint" ""
+		(property "Footprint" "Capacitor_SMD:C_0402_1005Metric"
 			(at 290.83 33.02 0)
 			(hide yes)
@@
 			)
 		)
-		(property "Footprint" ""
+		(property "Footprint" "Capacitor_SMD:C_0402_1005Metric"
 			(at 387.35 190.5 0)
 			(hide yes)
@@
 			)
 		)
-		(property "Footprint" ""
+		(property "Footprint" "Capacitor_SMD:C_0402_1005Metric"
 			(at 300.99 33.02 0)
 			(hide yes)
@@
 			)
 		)
-		(property "Footprint" ""
+		(property "Footprint" "slate113:KEY-SMD_KMR2XXGXXX"
 			(at 34.29 83.82 0)
 			(hide yes)
@@
 			)
 		)
+		(property "Manufacturer" "C&K"
+			(at 34.29 83.82 0)
+			(hide yes)
+			(show_name no)
+			(do_not_autoplace no)
+			(effects
+				(font
+					(size 1.27 1.27)
+				)
+			)
+		)
+		(property "MPN" "KMR231GLFS"
+			(at 34.29 83.82 0)
+			(hide yes)
+			(show_name no)
+			(do_not_autoplace no)
+			(effects
+				(font
+					(size 1.27 1.27)
+				)
+			)
+		)
+		(property "LCSC Part" "C99271"
+			(at 34.29 83.82 0)
+			(hide yes)
+			(show_name no)
+			(do_not_autoplace no)
+			(effects
+				(font
+					(size 1.27 1.27)
+				)
+			)
+		)
 		(pin "1"
 		)
@@
 			)
 		)
-		(property "Footprint" ""
+		(property "Footprint" "slate113:KEY-SMD_KMR2XXGXXX"
 			(at 95.25 81.28 0)
 			(hide yes)
@@
 			(hide yes)
 			(show_name no)
+			(do_not_autoplace no)
+			(effects
+				(font
+					(size 1.27 1.27)
+				)
+			)
+		)
+		(property "Manufacturer" "C&K"
+			(at 95.25 81.28 0)
+			(hide yes)
+			(show_name no)
+			(do_not_autoplace no)
+			(effects
+				(font
+					(size 1.27 1.27)
+				)
+			)
+		)
+		(property "MPN" "KMR231GLFS"
+			(at 95.25 81.28 0)
+			(hide yes)
+			(show_name no)
+			(do_not_autoplace no)
+			(effects
+				(font
+					(size 1.27 1.27)
+				)
+			)
+		)
+		(property "LCSC Part" "C99271"
+			(at 95.25 81.28 0)
+			(hide yes)
+			(show_name no)
