File: slate113.kicad_pcb (KiCad board)
At the start: 8 copper layers, 586 parts, among them CN1 DF40C-50DP-0.4V, CN10 DF40C-40DP-0.4V, CN11 DF40C-30DP-0.4V, CN12 DF40C-50DS-0.4V, CN13 DF40C-50DS-0.4V, CN14 DF40C-30DP-0.4V, CN15 DF40C-24DS-0.4V, CN16 DF40C-24DS-0.4V, CN17 0530470310, CN18 DF40C-10DP-0.4V, CN19 DF40C-24DP-0.4V, CN2 DF40C-50DP-0.4V, CN20 DF40C-24DP-0.4V, CN21 DF40C-40DS-0.4V, CN22 DF40C-40DS-0.4V, CN3 DF40C-30DS-0.4V, CN4 DF40C-40DS-0.4V, CN5 DF40C-40DP-0.4V, CN6 DF40C-40DS-0.4V, CN7 DF40C-30DS-0.4V, CN8 DF40C-40DP-0.4V, CN9 DF40C-40DP-0.4V, J1 RFPC-SMA27-F, J10 Conn_Coaxial, J11 RFPC-SMA27-F, J12 Conn_Coaxial, J13 U.FL, J14 U.FL, J15 U.FL, J16 U.FL, J17 U.FL, J18 U.FL, J19 U.FL, J2 TYPE-C16PIN, J20 U.FL, J22 RFPC-SMA27-F, J23 RFPC-SMA27-F, J24 Conn_Coaxial, J25 RFPC-SMA27-F, J26 Conn_Coaxial, J3 Conn_Coaxial, J4 DF40C-100DP-0.4V51*2, J6 395-016-520-202, J7 Conn_Coaxial, J8 RFPC-SMA27-F, J9 Bus_M.2_Socket_B, Q1 MMBT3904-TP, Q4 MMBT3904-C20526, Q5 CSD17575Q3, Q6 CSD17575Q3, Q7 CSD17575Q3, Q8 CSD17575Q3, SW1 SW_Push, SW2 SW_Push, SW3 SW_Push, SW4 SW_Push, U1 FUSB302BMPX, U10 TS3A24159DGSR, U11 SiP32508DT, U12 PI3USB302-AZBEX, U13 W25Q32JVSSIQ, U14 SiP32508DT, U15 TS5A23157DGSR, U17 SiP32508DT, U18 GL3523-OTY3C, U19 TXM27.12M0004322DBBDO00T, U2 CH224K, U20 CC1101RGPR, U21 0896BM15A0001001E, U22 LC29HBA, U23 EM4095HMSO16B+, U24 PE4259-63, U25 PE4259-63, U26 PE4259-63, U27 PE4259-63, U28 0433BM15A0001001E, U29 PN7160A1HN/C100E, U3 BQ25792RQMR, U30 PE4259-63, U31 S2B-PH-K-S-GW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

Commit message: continued work on carrier board, started work on m.2 board
Parts:
- added H5: MountingHole_Pad, MountingHole:MountingHole_3.2mm_M3_Pad_Via, F.Cu at (232.0, 124.7)
- added H6: MountingHole_Pad, MountingHole:MountingHole_3.2mm_M3_Pad_Via, F.Cu at (232.0, 136.7)
- moved C109 473.5 mm to (410.9, 40.7)
- moved C110 473.5 mm to (309.9, 31.1)
- moved C112 473.5 mm to (410.9, 42.7)
- moved C113 473.5 mm to (309.9, 36.2)
- moved Card1 473.5 mm to (413.4, 124.2)
- moved R19 473.5 mm to (333.9, 31.1)
- moved R20 473.5 mm to (333.9, 33.7)
- moved R21 473.5 mm to (333.9, 36.2)
- moved R22 473.5 mm to (333.9, 38.7)
- moved R23 473.5 mm to (333.9, 41.2)
- moved R26 473.5 mm to (333.9, 46.2)
- moved R38 473.5 mm to (333.9, 76.3)
- moved R62 473.5 mm to (337.9, 63.8)
- moved R63 473.5 mm to (337.9, 66.3)
- moved R64 473.5 mm to (337.9, 68.8)
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Connections:
- CN10 pad 35: PCIE0_WAKE -> MODEM_WAKE
- CN10 pad 37: unconnected-(CN10-Pad37) -> MODEM_RESET_N
- CN4 pad 35: PCIE0_WAKE -> MODEM_WAKE
- CN4 pad 37: unconnected-(CN4-Pad37) -> MODEM_RESET_N
- CN6 pad 35: PCIE0_WAKE -> MODEM_WAKE
- CN6 pad 37: unconnected-(CN6-Pad37) -> MODEM_RESET_N
- CN9 pad 35: PCIE0_WAKE -> MODEM_WAKE
- CN9 pad 37: unconnected-(CN9-Pad37) -> MODEM_RESET_N
- J4 pad 51: unconnected-(J4-Pad51) -> MODEM_RESET_N
- J4 pad 55: unconnected-(J4-Pad55) -> MODEM_WAKE
- J9 pad 67: PCIE0_PERST -> MODEM_RESET_N
Routing:
- net RP_ACC_AUX1: track 0.00 -> 90.5 mm, vias 0 -> 5
- net RP_ACC_RESET_N: track 0.00 -> 53.4 mm, vias 0 -> 4
- net RP_ACC_CS0_N: track 0.00 -> 51.3 mm, vias 0 -> 4
- net RP_ACC_MOSI: track 0.00 -> 48.3 mm, vias 0 -> 3
- net MODEM_RESET_N: track 0.00 -> 39.6 mm
- net CM5_ACC_MISO: track 0.00 -> 35.5 mm, vias 0 -> 2
- net CM5_ACC_SCK: track 0.00 -> 33.9 mm, vias 0 -> 3
- net CM5_ACC_AUX0: track 0.00 -> 32.8 mm, vias 0 -> 3
- net CM5_ACC_IRQ0: track 0.00 -> 27.8 mm, vias 0 -> 3
- net GND: track 92.3 -> 117.3 mm, vias 31 -> 41
- net PCIE0_RXP: track 0.00 -> 23.8 mm
- net PCIE0_REFCLKP: track 0.00 -> 23.7 mm, vias 0 -> 2
- net PCIE0_TXN: track 0.00 -> 21.8 mm
- net PCIE0_RXN: track 0.00 -> 20.1 mm
- net PCIE0_TXP: track 0.00 -> 17.1 mm
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
Commit message: finished m.2 board and copper pours, completed antenna bracket and power board, finished slateconnect board, reorganized libraries
Parts:
- added R142: 50Ω, Resistor_SMD:R_0402_1005Metric, F.Cu at (170.5, 35.2)
- added R143: 50Ω, Resistor_SMD:R_0402_1005Metric, F.Cu at (185.4, 35.2)
- added R144: 50Ω, Resistor_SMD:R_0402_1005Metric, F.Cu at (110.6, 35.1)
- added R145: 50Ω, Resistor_SMD:R_0402_1005Metric, F.Cu at (125.6, 35.1)
- added R146: 50Ω, Resistor_SMD:R_0402_1005Metric, F.Cu at (140.4, 35.2)
- added R24: 50Ω, Resistor_SMD:R_0402_1005Metric, F.Cu at (155.5, 35.2)
- added REF**: MountingHole_2.1mm, MountingHole:MountingHole_2.1mm, F.Cu at (276.8, 24.4)
- added REF**: MountingHole_2.1mm, MountingHole:MountingHole_2.1mm, F.Cu at (208.1, 82.6)
- added REF**: MountingHole_2.1mm, MountingHole:MountingHole_2.1mm, F.Cu at (190.8, 29.0)
- added REF**: MountingHole_2.1mm, MountingHole:MountingHole_2.1mm, F.Cu at (278.3, 130.8)
- added REF**: MountingHole_2.1mm, MountingHole:MountingHole_2.1mm, F.Cu at (204.2, 24.4)
- added REF**: MountingHole_2.1mm, MountingHole:MountingHole_2.1mm, F.Cu at (100.1, 29.0)
- added REF**: MountingHole_2.1mm, MountingHole:MountingHole_2.1mm, F.Cu at (234.3, 66.1)
- added REF**: MountingHole_2.1mm, MountingHole:MountingHole_2.1mm, F.Cu at (204.2, 50.7)
- added REF**: MountingHole_2.1mm, MountingHole:MountingHole_2.1mm, F.Cu at (208.1, 95.2)
- added REF**: MountingHole_2.1mm, MountingHole:MountingHole_2.1mm, F.Cu at (63.8, 82.6)
- added REF**: MountingHole_2.1mm, MountingHole:MountingHole_2.1mm, F.Cu at (63.8, 95.2)
- added REF**: MountingHole_2.1mm, MountingHole:MountingHole_2.1mm, F.Cu at (100.1, 44.1)
- added REF**: MountingHole_2.1mm, MountingHole:MountingHole_2.1mm, F.Cu at (234.1, 130.8)
- added REF**: MountingHole_2.1mm, MountingHole:MountingHole_2.1mm, F.Cu at (276.9, 50.6)
- added REF**: MountingHole_2.1mm, MountingHole:MountingHole_2.1mm, F.Cu at (190.8, 44.1)
- C143, C144, C145, C146, C148, C149, C151, C152, C153, C154, C18, C20, CN5, D5, D6, D7, R134, R135, R136, R137, R138, R139, R140, R141, R30, R77, R78, R79, R80, R81, R82, R83, R84, R85, R86, R87, R88, R89, R90, R91, R92, R93, R94, R95, U10, U55, U56, U57, U58, U59, U60, U61: moved to B.Cu
- CN17: value 0530470310 -> 530480310
- moved C13 449.3 mm to (276.0, 38.7), turned to 90 degrees
- moved C11 446.3 mm to (268.9, 45.3)
- moved C14 440.5 mm to (269.1, 33.7), turned to -90 degrees
- moved C15 432.8 mm to (260.3, 38.5)
- moved C5 431.9 mm to (249.2, 41.7), turned to 90 degrees
- moved C17 431.2 mm to (263.6, 27.2), turned to 90 degrees
- moved C6 430.7 mm to (249.9, 38.9)
- moved C16 429.5 mm to (261.1, 27.2), turned to 90 degrees
- moved C12 426.0 mm to (253.5, 29.9)
- moved C10 424.5 mm to (250.1, 30.4), turned to 180 degrees
- moved C4 419.1 mm to (235.9, 37.6), turned to -90 degrees
- moved C7 418.9 mm to (237.6, 40.6), turned to 180 degrees
- moved C3 418.5 mm to (234.3, 37.6), turned to -90 degrees
- moved R11 408.7 mm to (272.2, 40.2)
- moved R12 407.3 mm to (272.2, 38.2)
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Connections:
- C13 pad 1: SW -> L3_BOOST
- C157 pad 2: PGND -> GND
- C3 pad 2: Net-(U3-REGN) -> REGN
- C6 pad 1: BATT -> VBAT
- CN10 pad 25: SD_VDD -> 3V3
- CN10 pad 38: unconnected-(CN10-Pad38) -> 1V8
- CN21 pad 14: SC_SEL0 -> unconnected-(CN21-Pad14)
- CN21 pad 15: SC_SEL1 -> unconnected-(CN21-Pad15)
- CN21 pad 16: SC_SEL2 -> unconnected-(CN21-Pad16)
- CN21 pad 17: SC_SEL3 -> unconnected-(CN21-Pad17)
- CN21 pad 18: SC_SEL4 -> unconnected-(CN21-Pad18)
- CN21 pad 19: SC_SEL5 -> unconnected-(CN21-Pad19)
- CN21 pad 20: SC_SEL6 -> unconnected-(CN21-Pad20)
- CN21 pad 21: SC_SEL7 -> unconnected-(CN21-Pad21)
- CN22 pad 14: SC_SEL0 -> unconnected-(CN22-Pad14)
- CN22 pad 15: SC_SEL1 -> unconnected-(CN22-Pad15)
- CN22 pad 16: SC_SEL2 -> unconnected-(CN22-Pad16)
- CN22 pad 17: SC_SEL3 -> unconnected-(CN22-Pad17)
- CN22 pad 18: SC_SEL4 -> unconnected-(CN22-Pad18)
- CN22 pad 19: SC_SEL5 -> unconnected-(CN22-Pad19)
- CN22 pad 20: SC_SEL6 -> unconnected-(CN22-Pad20)
- CN22 pad 21: SC_SEL7 -> unconnected-(CN22-Pad21)
- CN4 pad 25: SD_VDD -> 3V3
- CN4 pad 38: unconnected-(CN4-Pad38) -> 1V8
- CN5 pad 14: SC_SEL0 -> unconnected-(CN5-Pad14)
- CN5 pad 15: SC_SEL1 -> unconnected-(CN5-Pad15)
- CN5 pad 16: SC_SEL2 -> unconnected-(CN5-Pad16)
- CN5 pad 17: SC_SEL3 -> unconnected-(CN5-Pad17)
- CN5 pad 18: SC_SEL4 -> unconnected-(CN5-Pad18)
- CN5 pad 19: SC_SEL5 -> unconnected-(CN5-Pad19)
- CN5 pad 20: SC_SEL6 -> unconnected-(CN5-Pad20)
- CN5 pad 21: SC_SEL7 -> unconnected-(CN5-Pad21)
- CN6 pad 25: SD_VDD -> 3V3
- CN6 pad 38: unconnected-(CN6-Pad38) -> 1V8
- CN8 pad 14: SC_SEL0 -> unconnected-(CN8-Pad14)
- CN8 pad 15: SC_SEL1 -> unconnected-(CN8-Pad15)
- CN8 pad 16: SC_SEL2 -> unconnected-(CN8-Pad16)
- CN8 pad 17: SC_SEL3 -> unconnected-(CN8-Pad17)
- CN8 pad 18: SC_SEL4 -> unconnected-(CN8-Pad18)
- CN8 pad 19: SC_SEL5 -> unconnected-(CN8-Pad19)
- CN8 pad 20: SC_SEL6 -> unconnected-(CN8-Pad20)
- CN8 pad 21: SC_SEL7 -> unconnected-(CN8-Pad21)
- CN9 pad 25: SD_VDD -> 3V3
- CN9 pad 38: unconnected-(CN9-Pad38) -> 1V8
- J2 pad A6: J2_DP -> unconnected-(J2-DP1-PadA6)
- J2 pad A7: J2_DN -> unconnected-(J2-DN1-PadA7)
- J2 pad B6: J2_DP -> unconnected-(J2-DP2-PadB6)
- J2 pad B7: J2_DN -> unconnected-(J2-DN2-PadB7)
- L2 pad 1: Net-(U3-SW1) -> SW1
- L2 pad 2: Net-(U3-SW2) -> SW2
- R14 pad 2: VOUT -> CM5_5V
- U2 pad 5: J2_DN -> unconnected-(U2-DM-Pad5)
- U3 pad 18: BATT -> VBAT
- U3 pad 22: BATT -> VBAT
- U3 pad 23: BATT -> VBAT
- U3 pad 26: Net-(U3-SW2) -> SW2
- U3 pad 28: Net-(U3-SW1) -> SW1
- U3 pad 5: Net-(U3-REGN) -> REGN
- U6 pad 12: LCD_LEDK -> LCD_LED_K
- U6 pad 13: LCD_LEDK -> LCD_LED_K
Routing:
- net VIN_EXT: track 63.8 -> 331.5 mm, vias 6 -> 14
- net VBUS: track 74.4 -> 297.8 mm, vias 7 -> 11
- net 3V3: track 20.3 -> 215.1 mm, vias 7 -> 32
- net GND: track 117.3 -> 282.9 mm, vias 41 -> 163
- net SC_POWER_STAT: track 0.00 -> 136.4 mm, vias 0 -> 6
- net SC_SINK_EN: track 0.00 -> 125.8 mm, vias 0 -> 5
- net CM5_ACC_CS0_N: track 38.6 -> 161.7 mm, vias 3 -> 6
- net SC_SOURCE_EN: track 0.00 -> 118.7 mm, vias 0 -> 2
- net RP_ACC_CS0_N: track 51.3 -> 162.8 mm, vias 4 -> 6
- net RP_ACC_MISO: track 0.00 -> 110.9 mm, vias 0 -> 4
- net CM5_ACC_MISO: track 35.5 -> 144.2 mm, vias 2 -> 5
- net RP_ACC_MOSI: track 48.3 -> 155.2 mm, vias 3 -> 5
- net CM5_ACC_MOSI: track 40.5 -> 143.0 mm, vias 3 -> 5
- net RP_ACC_SCK: track 0.98 -> 103.3 mm, vias 1 -> 5
- net SC_ID_SCL: track 0.00 -> 100.8 mm, vias 0 -> 3
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- added copper zone on In2.Cu, net 3V3
- added copper zone on In2.Cu, net M2_3V3
- removed copper zone on In4.Cu, net 3V3
Other:
- board outline added: 220.6 x 112.5 mm
