File: Kicad Project/slate113.kicad_pcb (KiCad board)
At the start: 8 copper layers, 220.6 x 112.5 mm, 609 parts, among them CN1 DF40C-50DP-0.4V, CN10 DF40C-40DP-0.4V, CN11 DF40C-30DP-0.4V, CN12 DF40C-50DS-0.4V, CN13 DF40C-50DS-0.4V, CN14 DF40C-30DP-0.4V, CN15 DF40C-24DS-0.4V, CN16 DF40C-24DS-0.4V, CN17 530480310, CN18 DF40C-10DP-0.4V, CN19 DF40C-24DP-0.4V, CN2 DF40C-50DP-0.4V, CN20 DF40C-24DP-0.4V, CN21 DF40C-40DS-0.4V, CN22 DF40C-40DS-0.4V, CN3 DF40C-30DS-0.4V, CN4 DF40C-40DS-0.4V, CN5 DF40C-40DP-0.4V, CN6 DF40C-40DS-0.4V, CN7 DF40C-30DS-0.4V, CN8 DF40C-40DP-0.4V, CN9 DF40C-40DP-0.4V, J1 RFPC-SMA27-F, J10 Conn_Coaxial, J11 RFPC-SMA27-F, J12 Conn_Coaxial, J13 U.FL, J14 U.FL, J15 U.FL, J16 U.FL, J17 U.FL, J18 U.FL, J19 U.FL, J2 TYPE-C16PIN, J20 U.FL, J22 RFPC-SMA27-F, J23 RFPC-SMA27-F, J24 Conn_Coaxial, J25 RFPC-SMA27-F, J26 Conn_Coaxial, J3 Conn_Coaxial, J4 DF40C-100DP-0.4V51*2, J6 395-016-520-202, J7 Conn_Coaxial, J8 RFPC-SMA27-F, J9 Bus_M.2_Socket_B, Q1 MMBT3904-TP, Q4 MMBT3904-C20526, Q5 CSD17575Q3, Q6 CSD17575Q3, Q7 CSD17575Q3, Q8 CSD17575Q3, SW1 SW_Push, SW2 SW_Push, SW3 SW_Push, SW4 SW_Push, U1 FUSB302BMPX, U10 TS3A24159DGSR, U11 SiP32508DT, U12 PI3USB302-AZBEX, U13 W25Q32JVSSIQ, U14 SiP32508DT, U15 TS5A23157DGSR, U17 SiP32508DT, U18 GL3523-OTY3C, U19 TXM27.12M0004322DBBDO00T, U2 CH224K, U20 CC1101RGPR, U21 0896BM15A0001001E, U22 LC29HBA, U23 EM4095HMSO16B+, U24 PE4259-63, U25 PE4259-63, U26 PE4259-63, U27 PE4259-63, U28 0433BM15A0001001E, U29 PN7160A1HN/C100E, U3 BQ25792RQMR, U30 PE4259-63, U31 S2B-PH-K-S-GW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

Commit message: organized repo, added license, and readme
Parts:
- moved C230 537.9 mm to (474.1, 57.6)
- moved C231 537.9 mm to (474.1, 59.6)
- moved C232 537.9 mm to (474.1, 61.6)
- moved C233 537.9 mm to (474.1, 63.6)
- moved C234 537.9 mm to (474.1, 65.5)
- moved C25 537.9 mm to (358.1, 54.0)
- moved C28 537.9 mm to (468.3, 53.7)
- moved C29 537.9 mm to (468.3, 55.7)
- moved C35 537.9 mm to (468.3, 57.6)
- moved C58 537.9 mm to (362.1, 69.0)
- moved C60 537.9 mm to (468.3, 59.6)
- moved C63 537.9 mm to (362.1, 79.1)
- moved C64 537.9 mm to (468.3, 61.6)
- moved C65 537.9 mm to (468.3, 63.6)
- moved C66 537.9 mm to (468.3, 65.5)
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Connections:
- C58 pad 2: 3V3 -> GPS_VCC
- R104 pad 1: 3V3 -> GPS_VCC
- R132 pad 2: 3V3 -> GPS_VCC
- R133 pad 1: 3V3 -> GPS_VCC
- U33 pad 2: 3V3 -> GPS_VCC
- U64 pad 24: 3V3 -> GPS_VCC
Routing:
- net GPS_UART_TX: track 0.00 -> 63.8 mm, vias 0 -> 2
- net BOOT: track 0.00 -> 55.6 mm
- net RP_ACC_MOSI: track 155.2 -> 207.6 mm, vias 5 -> 7
- net GPS_WAKEUP: track 0.00 -> 47.9 mm, vias 0 -> 2
- net RP_ACC_MISO: track 110.9 -> 154.8 mm, vias 4 -> 6
- net GPS_WI: track 0.00 -> 42.8 mm
- net LED_DATA_3V3: track 0.00 -> 42.4 mm, vias 0 -> 2
- net RP_ACC_SCK: track 103.3 -> 145.4 mm, vias 5 -> 7
- net GPS_1PPS: track 0.00 -> 39.9 mm, vias 0 -> 2
- net RP_ACC_IRQ0: track 48.3 -> 87.8 mm, vias 2 -> 4
- net RADIO_SPI0_MOSI: track 0.00 -> 35.3 mm, vias 0 -> 2
- net BADUSB_DP: track 0.00 -> 34.8 mm, vias 0 -> 2
- net RADIO_SPI0_MISO: track 0.00 -> 34.4 mm, vias 0 -> 2
- net BADUSB_DM: track 0.00 -> 34.1 mm, vias 0 -> 2
- net RADIO_SPI0_SCK: track 0.00 -> 33.7 mm, vias 0 -> 2
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Other:
- board size 220.6 x 112.5 mm -> 212.7 x 112.5 mm

Commit message: updated radio schematic, updated slate113 pcb, updated project file
Parts:
- added C236: 100nF, Capacitor_SMD:C_0603_1608Metric, F.Cu at (148.2, 116.3)
- added C237: 220pF, Capacitor_SMD:C_0402_1005Metric, F.Cu at (161.0, 121.5)
- added C238: 220pF, Capacitor_SMD:C_0402_1005Metric, F.Cu at (161.0, 120.2)
- added C239: 1µF, Capacitor_SMD:C_0603_1608Metric, F.Cu at (149.9, 116.3)
- added C240: 10nF, Capacitor_SMD:C_0603_1608Metric, F.Cu at (153.2, 116.3)
- added C241: 220pF, Capacitor_SMD:C_0402_1005Metric, F.Cu at (161.0, 119.0)
- added C242: 10nF, Capacitor_SMD:C_0603_1608Metric, F.Cu at (151.6, 116.3)
- moved C233 365.7 mm to (116.7, 141.0), turned to 90 degrees
- moved C234 364.5 mm to (117.0, 138.7), turned to 180 degrees
- moved U72 360.8 mm to (119.0, 140.9)
- moved Y3 327.0 mm to (157.6, 127.7), turned to 180 degrees
- moved C28 323.0 mm to (153.7, 126.9), turned to 90 degrees
- moved C29 317.2 mm to (158.8, 125.1), turned to 180 degrees
- moved U64 311.9 mm to (141.6, 118.7)
- moved R132 279.5 mm to (132.8, 115.7), turned to 180 degrees
- moved R133 279.0 mm to (132.8, 113.9)
- moved U26 264.3 mm to (165.3, 121.1), turned to 180 degrees
- moved U27 264.2 mm to (165.3, 125.4), turned to 180 degrees
- moved C96 250.2 mm to (123.4, 147.5), turned to 180 degrees
- moved C95 246.8 mm to (126.9, 144.7), turned to 90 degrees
- moved R39 234.3 mm to (160.5, 117.4), turned to 180 degrees
- moved C25 219.6 mm to (149.8, 123.8)
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Connections:
- U20 pad 11: CC1101_CAPS -> AVDD11_CAP
- U20 pad 14: CC1101_CAPS -> AVDD14_CAP
- U20 pad 15: CC1101_CAPS -> AVDD15_CAP
- U20 pad 18: GND -> Net-(U20-DGUARD)
- U20 pad 9: CC1101_CAPS -> AVDD9_CAP
- U33 pad 8: GPS_UART_TX -> GPS_UART_RX
- U33 pad 9: GPS_UART_RX -> GPS_UART_TX
- U72 pad 3: CM5_UART_TX -> GPS_UART_RX
Routing:
- net GPS_UART_RX_F: track 0.00 -> 74.3 mm, vias 0 -> 3
- net VDD_EXT: track 0.00 -> 62.6 mm, vias 0 -> 3
- net RADIO_I2C0_SDA: track 19.7 -> 60.3 mm, vias 3 -> 5
- net BAND_SEL_1: track 0.00 -> 36.4 mm, vias 0 -> 3
- net GPS_VCC: track 2.48 -> 31.7 mm, vias 1 -> 8
- net RADIO_I2C0_SCL: track 22.7 -> 47.9 mm
- net GND: track 303.7 -> 326.7 mm, vias 191 -> 212
- net RADIO_EN: track 0.00 -> 21.7 mm, vias 0 -> 2
- net AVDD14_CAP: track 0.00 -> 12.1 mm
- net RF_N: track 0.00 -> 11.7 mm, vias 0 -> 2
- net AVDD9_CAP: track 0.00 -> 11.1 mm, vias 0 -> 2
- net RF_P: track 0.00 -> 10.1 mm, vias 0 -> 2
- net GPS_UART_RX: track 3.04 -> 12.6 mm, vias 0 -> 2
- net Net-(U20-DGUARD): track 0.00 -> 8.12 mm, vias 0 -> 2
- net Net-(C96-Pad2): track 0.00 -> 6.35 mm
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- added copper zone on In2.Cu, net GPS_VCC
