File: Kicad Project/slate113.kicad_pcb (KiCad board)
At the start: 8 copper layers, 212.7 x 112.5 mm, 616 parts, among them CN1 DF40C-50DP-0.4V, CN10 DF40C-40DP-0.4V, CN11 DF40C-30DP-0.4V, CN12 DF40C-50DS-0.4V, CN13 DF40C-50DS-0.4V, CN14 DF40C-30DP-0.4V, CN15 DF40C-24DS-0.4V, CN16 DF40C-24DS-0.4V, CN17 530480310, CN18 DF40C-10DP-0.4V, CN19 DF40C-24DP-0.4V, CN2 DF40C-50DP-0.4V, CN20 DF40C-24DP-0.4V, CN21 DF40C-40DS-0.4V, CN22 DF40C-40DS-0.4V, CN3 DF40C-30DS-0.4V, CN4 DF40C-40DS-0.4V, CN5 DF40C-40DP-0.4V, CN6 DF40C-40DS-0.4V, CN7 DF40C-30DS-0.4V, CN8 DF40C-40DP-0.4V, CN9 DF40C-40DP-0.4V, J1 RFPC-SMA27-F, J10 Conn_Coaxial, J11 RFPC-SMA27-F, J12 Conn_Coaxial, J13 U.FL, J14 U.FL, J15 U.FL, J16 U.FL, J17 U.FL, J18 U.FL, J19 U.FL, J2 TYPE-C16PIN, J20 U.FL, J22 RFPC-SMA27-F, J23 RFPC-SMA27-F, J24 Conn_Coaxial, J25 RFPC-SMA27-F, J26 Conn_Coaxial, J3 Conn_Coaxial, J4 DF40C-100DP-0.4V51*2, J6 395-016-520-202, J7 Conn_Coaxial, J8 RFPC-SMA27-F, J9 Bus_M.2_Socket_B, Q1 MMBT3904-TP, Q4 MMBT3904-C20526, Q5 CSD17575Q3, Q6 CSD17575Q3, Q7 CSD17575Q3, Q8 CSD17575Q3, SW1 SW_Push, SW2 SW_Push, SW3 SW_Push, SW4 SW_Push, U1 FUSB302BMPX, U10 TS3A24159DGSR, U11 SiP32508DT, U12 PI3USB302-AZBEX, U13 W25Q32JVSSIQ, U14 SiP32508DT, U15 TS5A23157DGSR, U17 SiP32508DT, U18 GL3523-OTY3C, U19 TXM27.12M0004322DBBDO00T, U2 CH224K, U20 CC1101RGPR, U21 0896BM15A0001001E, U22 LC29HBA, U23 EM4095HMSO16B+, U24 PE4259-63, U25 PE4259-63, U26 PE4259-63, U27 PE4259-63, U28 0433BM15A0001001E, U29 PN7160A1HN/C100E, U3 BQ25792RQMR, U30 PE4259-63, U31 S2B-PH-K-S-GW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

Commit message: added devlog and worked on NFC stack
Parts:
- moved R114 281.6 mm to (125.4, 117.3), turned to 180 degrees
- moved C68 243.5 mm to (120.8, 116.6)
- moved C69 243.4 mm to (120.8, 118.5)
- moved C71 243.0 mm to (120.8, 120.1)
- moved C76 239.7 mm to (123.3, 124.7)
- moved C72 237.6 mm to (125.4, 114.0)
- moved C74 237.3 mm to (125.4, 115.6)
Routing:
- net GPS_VCC: track 31.7 -> 81.6 mm, vias 8 -> 14
- net NFC_VEN: track 0.00 -> 43.1 mm, vias 0 -> 3
- net NFC_VDDTX: track 0.00 -> 19.9 mm
- net GND: track 326.7 -> 336.5 mm, vias 212 -> 220

Commit message: wired up NFC, RFID, and GPS systems
Parts:
- removed U32: S2B-PH-K-S-GW, slate113:CONN-TH_S2B-PH-K-S-GW
- added C243: 100nF, Capacitor_SMD:C_0402_1005Metric, B.Cu at (146.4, 118.8)
- added C244: 1nF, Capacitor_SMD:C_0603_1608Metric, F.Cu at (124.2, 123.1)
- added C245: 1nF, Capacitor_SMD:C_0603_1608Metric, B.Cu at (132.6, 119.3)
- added C246: 100nF, Capacitor_SMD:C_0402_1005Metric, B.Cu at (144.4, 125.5)
- added L11: YSPIT0520A-R16M, slate113:IND-SMD_L5.5-W5.3, B.Cu at (143.3, 118.5)
- added L12: YSPIT0520A-R16M, slate113:IND-SMD_L5.5-W5.3, B.Cu at (139.9, 124.5)
- added R147: 1.5Ω, Resistor_SMD:R_1206_3216Metric, B.Cu at (138.4, 118.2)
- added R148: 2.7Ω, Resistor_SMD:R_1206_3216Metric, B.Cu at (126.0, 128.2)
- added R149: 2.2kΩ, Capacitor_SMD:C_0603_1608Metric, B.Cu at (132.6, 117.5)
- added R150: 2.2kΩ, Capacitor_SMD:C_0603_1608Metric, B.Cu at (132.7, 124.8)
- added R151: 1.5Ω, Resistor_SMD:R_1206_3216Metric, B.Cu at (139.3, 128.9)
- added R152: 2.7Ω, Resistor_SMD:R_1206_3216Metric, B.Cu at (131.0, 128.9)
- added U73: B2B-PH-K-S, slate113:CONN-TH_B2B-PH-K-S, B.Cu at (164.7, 129.3)
- C35, C66: value 20pF -> 15pF; moved to B.Cu
- C75, C79, U19: moved to B.Cu
- U31: value S2B-PH-K-S-GW -> B2B-PH-K-S; footprint slate113:CONN-TH_S2B-PH-K-S-GW -> slate113:CONN-TH_B2B-PH-K-S
- moved U19 363.7 mm to (122.3, 129.3), turned to 180 degrees
- moved C35 354.0 mm to (120.2, 121.6), turned to 180 degrees
- moved C66 352.5 mm to (120.9, 124.8), turned to -90 degrees
- moved U35 341.5 mm to (127.9, 149.2)
- moved D2 308.0 mm to (170.8, 147.0), turned to 90 degrees
- moved Q1 304.5 mm to (167.5, 141.1)
- moved L8 303.1 mm to (169.5, 138.7), turned to 180 degrees
- moved C82 302.1 mm to (177.8, 125.3)
- moved U71 278.6 mm to (173.7, 126.4)
- moved D3 269.1 mm to (183.4, 125.0)
- moved D4 269.1 mm to (183.4, 127.2)
- moved R112 259.7 mm to (149.9, 133.1), turned to 90 degrees
- moved C88 253.5 mm to (123.3, 141.6), turned to 180 degrees
- moved R44 249.2 mm to (164.7, 141.0), turned to -90 degrees
- moved J20 246.3 mm to (175.8, 150.0), turned to -90 degrees
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Routing:
- net 3V3: track 219.6 -> 330.2 mm, vias 35 -> 40
- net RF_V2: track 0.00 -> 91.4 mm, vias 0 -> 5
- net RF_V1: track 0.00 -> 77.6 mm, vias 0 -> 4
- net GND: track 336.5 -> 401.4 mm, vias 220 -> 260
- net RADIO_5V: track 0.00 -> 45.1 mm, vias 0 -> 4
- net NFC_ANT2: track 0.00 -> 40.3 mm, vias 0 -> 2
- net GPS_RESET: track 0.00 -> 38.0 mm, vias 0 -> 3
- net 5V: track 0.00 -> 36.6 mm, vias 0 -> 2
- net NFC_ANT1: track 0.00 -> 29.7 mm, vias 0 -> 6
- net Net-(C243-Pad1): track 0.00 -> 28.3 mm, vias 0 -> 2
- net EM_SHD: track 0.00 -> 27.8 mm, vias 0 -> 4
- net NFC_XTAL1: track 0.00 -> 24.0 mm, vias 0 -> 4
- net NFC_VDDCORE: track 0.00 -> 22.7 mm, vias 0 -> 2
- net NFC_XTAL2: track 0.00 -> 22.3 mm, vias 0 -> 3
- net GPS_ANT: track 0.00 -> 21.1 mm, vias 0 -> 3
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