File: Kicad Project/io.kicad_sch (KiCad schematic)
At the start: 139 parts, among them CN1 DF40C-50DP-0.4V, J13 U.FL, J14 U.FL, J15 U.FL, J16 U.FL, J17 U.FL, J18 U.FL, U1 FUSB302BMPX, U12 PI3USB302-AZBEX, U13 W25Q32JVSSIQ, U14 SiP32508DT, U15 TS5A23157DGSR, U17 SiP32508DT, U18 GL3523-OTY3C, U30 PE4259-63, U36 PE4259-63, U37 CPL0605AT13R2455A, U38 X4C60K1-20SR, U39 XEC24P3-30GR, U40 AD8317ACPZ-R7, U41 AD8317ACPZ-R7, U42 AD8317ACPZ-R7, U43 LM339D, U53 SiP32508DT, U7 HD3SS3220RNHR, U70 SkyLab WG243, X1 X322525MOB4SI

Commit message: started work on IO
Connections:
- net FerriteGND: no longer USB1.25 (EH)
- net FerriteGND_IO: now also USB1.25 (EH)
Changed lines of the file:
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@@
 		)
 	)
-	(global_label "FerriteGND"
-		(shape input)
-		(at 132.08 92.71 180)
-		(fields_autoplaced yes)
-		(effects
-			(font
-				(size 1.27 1.27)
-			)
-			(justify right)
-		)
-		(property "Intersheetrefs" "${INTERSHEET_REFS}"
-			(at 119.0556 92.71 0)
-			(hide yes)
-			(show_name no)
-			(do_not_autoplace no)
-			(effects
-				(font
-					(size 1.27 1.27)
-				)
-				(justify right)
-			)
-		)
-	)
 	(global_label "GND"
 		(shape input)
@@
 			)
 		)
+	)
+	(global_label "FerriteGND_IO"
+		(shape input)
+		(at 132.08 92.71 0)
+		(fields_autoplaced yes)
+		(effects
+			(font
+				(size 1.27 1.27)
+			)
+			(justify left)
+		)
+		(property "Intersheetrefs" "${INTERSHEET_REFS}"
+			(at 148.0073 92.71 0)
+			(hide yes)
+			(show_name no)
+			(do_not_autoplace no)
+			(effects
+				(font
+					(size 1.27 1.27)
+				)
+				(justify left)
+			)
+		)

Commit message: worked on IO daughter board
Connections:
- net FerriteGND is gone; now on net FerriteGND_IO: RJ1.15 (SHELL), RJ1.16 (SHELL)

Commit message: made some schematic changes to power
Parts:
- removed C30, C31, C41: 100nF, Capacitor_SMD:C_0603_1608Metric, symbol Device:C_Small
- removed CN1: DF40C-50DP-0.4V, slate113:CONN-SMD_DF40C-50DP-0.4V, symbol slate113:DF40C-50DP-0.4V
- removed R34: 100kΩ, Resistor_SMD:R_0603_1608Metric, symbol Device:R_Small
- removed R35: 180kΩ, Resistor_SMD:R_0603_1608Metric, symbol Device:R_Small
- removed U12: PI3USB302-AZBEX, slate113:DHVQFN-20_L4.5-W2.5-P0.50-BL-EP, symbol slate113:PI3USB302-AZBEX
- removed U15: TS5A23157DGSR, slate113:MSOP-10_L3.0-W3.0-P0.50-LS5.0-BL, symbol slate113:TS5A23157DGSR
- removed U7: HD3SS3220RNHR, slate113:WQFN-30_L4.5-W2.5-P0.4-BL-EP, symbol slate113:HD3SS3220RNHR
- added C247, C248, C249, C250: 100nF, Capacitor_SMD:C_0603_1608Metric, symbol Device:C_Small
- added CN23: DF40C-60DP-0.4V, slate113:CONN-SMD_DF40C-60DP-0.4V, symbol slate113:DF40C-60DP-0.4V
Connections:
- net 2.4G_SENSE: now also CN23.24, CN23.37
- net 3V3: now also U1.3 (VDD), U1.4 (VDD), CN23.4, CN23.58; no longer C22.2, C23.2, C24.2
- net BLE_CTRL: now also CN23.38
- net BLE_SENSE: now also CN23.25
- net BT_EN: now also CN23.10
- net CM5_5V: now also U1.12 (VCONN), U1.13 (VCONN), CN23.3, CN23.59
- net COMBO_EN: now also CN23.50
- net ETH_MDI0N: now also CN23.57
- net ETH_MDI0P: now also CN23.5
- net ETH_MDI1N: now also CN23.56
- net ETH_MDI1P: now also CN23.7
- net ETH_MDI2N: now also CN23.6
- net ETH_MDI2P: now also CN23.55
- net ETH_MDI3N: now also CN23.54
- net ETH_MDI3P: now also CN23.8
- net FerriteGND_IO: now also CN23.61, CN23.62, CN23.63, CN23.64
- net GND: now also C1.2, C2.2, CN23.1, CN23.2, CN23.20, CN23.22, CN23.27, CN23.28, CN23.29, CN23.30, CN23.31, CN23.32, CN23.33, CN23.34, CN23.36, CN23.39, CN23.60
- net I2C0_SCL: now also CN23.19
- net I2C0_SDA: now also CN23.42
- net LAN0_GLED+: now also CN23.53
- net LAN0_YLED-: now also CN23.9
- net M2_DM: now also CN23.47
- net M2_DP: now also CN23.14
- net M2_EN: now also CN23.41
- net SBU1: now also CN23.18
- net SBU2: now also CN23.43
- net USB1_DN: now also CN23.26; no longer U18.26 (DM_P2)
- net USB1_DP: now also CN23.35; no longer U18.25 (DP_P2)
- net USB1_RX1N: now also CN23.12
- net USB1_RX1P: now also CN23.49; no longer USB1.A11 (RX2+)
- net USB1_RX2N: now also CN23.13
- net USB1_TX1N: now also C248.1
- net USB1_TX1P: now also C247.1
- net USB1_TX2N: now also C250.1
- net USB1_TX2P: now also C249.1
- net USB2_H_DM: now also CN23.40
- net USB2_H_DP: now also CN23.21
- net USBC1_INT_L: now also CN23.46
- net USB_HUB_EN: now also CN23.52
- net USB_HUB_RST: now also CN23.15
- net WIFI_CTRL: now also CN23.23
- net WIFI_EN: now also CN23.51
- net WOWLAN: now also CN23.11
- new net MUX_CAPS: C22.2, C23.2, C24.2
- new net USB1_RX2P: CN23.48, USB1.A11 (RX2+)
- new net USB1_TX1N_F: C248.2, CN23.16
- new net USB1_TX1P_F: C247.2, CN23.45
- new net USB1_TX2N_F: C250.2, CN23.17
- new net USB1_TX2P_F: C249.2, CN23.44
- no-connect marks 68 -> 56
Other:
- note removed: "1:2 Mux"
- note removed: "SBU Routing"
- note removed: "SS Mux (Not 1:2)"
- moved on the sheet: C1, C101, C2, C93, R45, R46, R47, R49, U40

Commit message: update schematics and flex cable project
Parts:
- added R124: 10kΩ, Resistor_SMD:R_0603_1608Metric, symbol Device:R_Small
Connections:
- net 3V3: now also R124.2
- net USB_HUB_EN: now also R124.1
Other:
- note added: "Random Resistor"
Changed lines of the file:
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@@
 	)
 	(rectangle
+		(start 167.894 88.9)
+		(end 189.23 137.414)
+		(stroke
+			(width 0)
+			(type default)
+		)
+		(fill
+			(type none)
+		)
+	)
+	(rectangle
 		(start 13.97 88.9)
 		(end 91.44 139.7)
@@
 		)
 	)
+	(text "Random Resistor\n"
+		(exclude_from_sim no)
+		(at 176.022 136.906 0)
+		(effects
+			(font
+				(size 1.27 1.27)
+			)
+		)
+	)
 	(text "Hub Flash\n"
 		(exclude_from_sim no)
@@
 		)
 	)
+	(global_label "3V3"
+		(shape input)
+		(at 180.34 107.95 90)
+		(fields_autoplaced yes)
+		(effects
+			(font
+				(size 1.27 1.27)
+			)
+			(justify left)
+		)
+		(property "Intersheetrefs" "${INTERSHEET_REFS}"
+			(at 180.34 101.4572 90)
+			(hide yes)
+			(show_name no)
+			(do_not_autoplace no)
+			(effects
+				(font
+					(size 1.27 1.27)
+				)
+				(justify left)
+			)
+		)
+	)
 	(global_label "GND"
 		(shape input)
@@
 		)
 	)
+	(global_label "USB_HUB_EN"
+		(shape input)
+		(at 180.34 113.03 270)
+		(fields_autoplaced yes)
+		(effects
+			(font
+				(size 1.27 1.27)
+			)
+			(justify right)
+		)
+		(property "Intersheetrefs" "${INTERSHEET_REFS}"
+			(at 180.34 128.1709 90)
+			(hide yes)
+			(show_name no)
+			(do_not_autoplace no)
+			(effects
+				(font
+					(size 1.27 1.27)
+				)
+				(justify right)
+			)
+		)
+	)
 	(global_label "GND"
 		(shape input)
@@
 					(unit 1)
 				)
+			)
+		)
+	)
+	(symbol
+		(lib_id "Device:R_Small")
+		(at 180.34 110.49 180)
+		(unit 1)
+		(body_style 1)
+		(exclude_from_sim no)
+		(in_bom yes)
+		(on_board yes)
+		(in_pos_files yes)
+		(dnp no)
+		(fields_autoplaced yes)
+		(property "Reference" "R124"
+			(at 175.26 110.49 90)
+			(show_name no)
+			(do_not_autoplace no)
+			(effects
+				(font
+					(size 1.016 1.016)
+				)
+			)
+		)
+		(property "Value" "10kΩ"
+			(at 177.8 110.49 90)
+			(show_name no)
+			(do_not_autoplace no)
+			(effects
+				(font
+					(size 1.27 1.27)
+				)
+			)
+		)
+		(property "Footprint" "Resistor_SMD:R_0603_1608Metric"
+			(at 180.34 110.49 0)
+			(hide yes)
+			(show_name no)
+			(do_not_autoplace no)
+			(effects
+				(font
+					(size 1.27 1.27)
+				)
+			)
+		)
+		(property "Datasheet" ""
+			(at 180.34 110.49 0)
+			(hide yes)
+			(show_name no)
+			(do_not_autoplace no)
+			(effects
+				(font
+					(size 1.27 1.27)
+				)
+			)
+		)
+		(property "Description" "Resistor, small symbol"
+			(at 180.34 110.49 0)
+			(hide yes)
+			(show_name no)
+			(do_not_autoplace no)
+			(effects
+				(font
+					(size 1.27 1.27)
+				)
+			)
+		)
+		(pin "1"
+		)
+		(pin "2"
+		)
+		(instances
+			(project "slate113"
+				(path "/d9c968d6-de70-422d-aa76-11643c5e786e"
+					(reference "R124")
+					(unit 1)
+				)
