File: Kicad Project/main_board.kicad_sch (KiCad schematic)
At the start: 100 parts, among them CN10 DF40C-40DP-0.4V, CN11 DF40C-30DP-0.4V, CN19 DF40C-24DP-0.4V, CN2 DF40C-50DP-0.4V, CN8 DF40C-40DP-0.4V, J4 DF40C-100DP-0.4V51*2, Q4 MMBT3904-C20526, SW1 SW_Push, SW2 SW_Push, U11 SiP32508DT, U47 ES8388, U48 TS5A23157DGSR, U49 TS5A23157DGSR, U50 PAM8302AASCR, U51 PAM8302AASCR, U52 TPS7A0233PDBVR, U62 PCA9306DCUR, U63 AP2120N-2.8TRG1, U65 MSM381ADB001, U66 DF40B-10DS-0.4V, U67 SIP32508DT-T1-GE3, U68 SN74AHCT125PWR, U69 TCA9535PWR, U8 ESD7104MUTAG_C2987068

Commit message: finished up the Slate Connect + M.2 board connectors on carrier, started work on the radio carrier connector
Connections:
- net 5V is gone; now on net CM5_5V: CN19.12
- net MODEM_W_DISABLE: now also U69.13 (P10)
- net R_UNUSED: no longer U69.13 (P10)
- no-connect marks 94 -> 99
Changed lines of the file:
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@@
 	)
 	(junction
-		(at 394.97 138.43)
-		(diameter 0)
-		(color 0 0 0 0)
-	)
-	(junction
 		(at 135.89 285.75)
 		(diameter 0)
@@
 	)
 	(junction
-		(at 397.51 138.43)
+		(at 229.87 340.36)
 		(diameter 0)
 		(color 0 0 0 0)
 	)
 	(junction
-		(at 229.87 340.36)
+		(at 135.89 271.78)
 		(diameter 0)
 		(color 0 0 0 0)
 	)
 	(junction
-		(at 135.89 271.78)
+		(at 261.62 133.35)
 		(diameter 0)
 		(color 0 0 0 0)
 	)
 	(junction
-		(at 261.62 133.35)
+		(at 394.97 138.43)
 		(diameter 0)
 		(color 0 0 0 0)
@@
 	)
 	(no_connect
+		(at 179.07 128.27)
+	)
+	(no_connect
 		(at 176.53 208.28)
 	)
@@
 	)
 	(no_connect
+		(at 184.15 128.27)
+	)
+	(no_connect
 		(at 133.35 177.8)
 	)
@@
 	)
 	(no_connect
+		(at 156.21 128.27)
+	)
+	(no_connect
 		(at 311.15 267.97)
 	)
@@
 	)
 	(no_connect
+		(at 134.62 318.77)
+	)
+	(no_connect
 		(at 204.47 208.28)
 	)
@@
 	)
 	(no_connect
+		(at 161.29 128.27)
+	)
+	(no_connect
 		(at 193.04 339.09)
 	)
@@
 	(wire
 		(pts
-			(xy 382.27 135.89) (xy 382.27 139.7)
-		)
-		(stroke
-			(width 0)
-			(type default)
-		)
-	)
-	(wire
-		(pts
 			(xy 384.81 138.43) (xy 384.81 139.7)
 		)
@@
 	(wire
 		(pts
-			(xy 379.73 134.62) (xy 379.73 139.7)
+			(xy 379.73 135.89) (xy 379.73 139.7)
 		)
 		(stroke
@@
 		)
 	)
+	(wire
+		(pts
+			(xy 382.27 137.16) (xy 382.27 139.7)
+		)
+		(stroke
+			(width 0)
+			(type default)
+		)
+	)
 	(polyline
 		(pts
@@
 	(wire
 		(pts
+			(xy 403.86 139.7) (xy 403.86 149.86)
+		)
+		(stroke
+			(width 0)
+			(type default)
+		)
+	)
+	(wire
+		(pts
 			(xy 444.5 335.28) (xy 444.5 337.82)
 		)
@@
 	(wire
 		(pts
-			(xy 397.51 138.43) (xy 397.51 139.7)
-		)
-		(stroke
-			(width 0)
-			(type default)
-		)
-	)
-	(wire
-		(pts
 			(xy 382.27 337.82) (xy 391.16 337.82)
 		)
@@
 	(wire
 		(pts
-			(xy 405.13 144.78) (xy 402.59 144.78)
+			(xy 405.13 144.78) (xy 401.32 144.78)
 		)
 		(stroke
@@
 	(wire
 		(pts
-			(xy 402.59 135.89) (xy 382.27 135.89)
+			(xy 401.32 137.16) (xy 382.27 137.16)
 		)
 		(stroke
@@
 	(wire
 		(pts
+			(xy 394.97 133.35) (xy 394.97 138.43)
+		)
+		(stroke
+			(width 0)
+			(type default)
+		)
+	)
+	(wire
+		(pts
 			(xy 397.51 162.56) (xy 397.51 160.02)
 		)
@@
 	(wire
 		(pts
+			(xy 403.86 139.7) (xy 397.51 139.7)
+		)
+		(stroke
+			(width 0)
+			(type default)
+		)
+	)
+	(wire
+		(pts
 			(xy 374.65 132.08) (xy 374.65 139.7)
 		)
@@
 	(wire
 		(pts
-			(xy 391.16 327.66) (xy 400.05 327.66)
+			(xy 397.51 133.35) (xy 394.97 133.35)
 		)
 		(stroke
@@
 	(wire
 		(pts
-			(xy 397.51 138.43) (xy 401.32 138.43)
+			(xy 391.16 327.66) (xy 400.05 327.66)
 		)
 		(stroke
@@
 	(wire
 		(pts
-			(xy 405.13 134.62) (xy 379.73 134.62)
+			(xy 405.13 135.89) (xy 379.73 135.89)
 		)
 		(stroke
@@
 	(wire
 		(pts
-			(xy 405.13 142.24) (xy 405.13 134.62)
+			(xy 405.13 142.24) (xy 405.13 135.89)
 		)
 		(stroke
@@
 	(wire
 		(pts
-			(xy 394.97 138.43) (xy 397.51 138.43)
-		)
-		(stroke
-			(width 0)
-			(type default)
-		)
-	)
-	(wire
-		(pts
 			(xy 238.76 300.99) (xy 240.03 300.99)
 		)
@@
 	(wire
 		(pts
-			(xy 402.59 144.78) (xy 402.59 135.89)
+			(xy 401.32 144.78) (xy 401.32 137.16)
 		)
 		(stroke
@@
 	(global_label "R_UNUSED"
 		(shape input)
-		(at 401.32 138.43 0)
+		(at 397.51 133.35 0)
 		(fields_autoplaced yes)
 		(effects
@@
 		)
 		(property "Intersheetrefs" "${INTERSHEET_REFS}"
-			(at 414.1628 138.43 0)
+			(at 410.3528 133.35 0)
 			(hide yes)
 			(show_name no)
@@
 		)
 	)
+	(global_label "MODEM_W_DISABLE"
+		(shape input)
+		(at 403.86 149.86 270)
+		(fields_autoplaced yes)
+		(effects
+			(font
+				(size 1.27 1.27)
+			)
+			(justify right)
+		)
+		(property "Intersheetrefs" "${INTERSHEET_REFS}"
+			(at 403.86 170.5041 90)
+			(hide yes)
+			(show_name no)
+			(do_not_autoplace no)
+			(effects
+				(font
+					(size 1.27 1.27)
+				)
+				(justify right)
+			)
+		)
+	)
 	(global_label "ETH_MDI1N"
 		(shape input)
@@
 		)
 	)
-	(global_label "5V"
+	(global_label "CM5_5V"
 		(shape input)
 		(at 132.08 318.77 0)
@@
 		)
 		(property "Intersheetrefs" "${INTERSHEET_REFS}"
-			(at 137.3633 318.77 0)
+			(at 142.2618 318.77 0)
 			(hide yes)
 			(show_name no)
@@
 		(in_pos_files yes)
 		(dnp no)
-		(fields_autoplaced yes)
 		(property "Reference" "U69"
-			(at 401.32 148.5899 90)
+			(at 364.744 144.78 0)
 			(show_name no)
 			(do_not_autoplace no)
@@
 		)
 		(property "Value" "TCA9535PWR"
-			(at 401.32 151.1299 90)
+			(at 362.204 144.78 0)
 			(show_name no)
 			(do_not_autoplace no)

Commit message: worked on the carrier board more and finish up the radio b2b connector (excluding LED stuff)
Connections:
- no-connect marks 99 -> 98
Changed lines of the file:
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@@
-	)
-	(no_connect
-		(at 134.62 318.77)
 	)
 	(no_connect

Commit message: finished carrier!
Parts:
- removed R121, R123, R125: 10kΩ, Resistor_SMD:R_0603_1608Metric, symbol Device:R_Small
Other:
- moved on the sheet: R122, R126, R127, R128, R129

Commit message: made some schematic changes to power
Parts:
- removed CN2: DF40C-50DP-0.4V, slate113:CONN-SMD_DF40C-50DP-0.4V, symbol slate113:DF40C-50DP-0.4V
- added CN24: DF40C-60DP-0.4V, slate113:CONN-SMD_DF40C-60DP-0.4V, symbol slate113:DF40C-60DP-0.4V
Connections:
- net 2.4G_SENSE: now also CN24.37
- net 3V3: now also CN24.4, CN24.58
- net 5G_SENSE: now also CN24.24
- net BLE_CTRL: now also CN24.38
- net BLE_SENSE: now also CN24.25
- net BT_EN: now also CN24.10
- net CM5_5V: now also CN24.3, CN24.59
- net COMBO_EN: now also CN24.50
- net ETH_MDI0N: now also CN24.57
- net ETH_MDI0P: now also CN24.5
- net ETH_MDI1N: now also CN24.56
- net ETH_MDI1P: now also CN24.7
- net ETH_MDI2N: now also CN24.6
- net ETH_MDI2P: now also CN24.55
- net ETH_MDI3N: now also CN24.54
- net ETH_MDI3P: now also CN24.8
- net GND: now also CN24.1, CN24.2, CN24.20, CN24.22, CN24.27, CN24.28, CN24.29, CN24.30, CN24.31, CN24.32, CN24.33, CN24.34, CN24.36, CN24.39, CN24.60
- net I2C0_SCL: now also CN24.19
- net I2C0_SDA: now also CN24.42
- net LAN0_GLED+: now also CN24.53
- net LAN0_YLED-: now also CN24.9
- net M2_DM: now also CN24.47
- net M2_DP: now also CN24.14
- net M2_EN: now also CN24.41
- net USB2_H_DM: now also CN24.40
- net USB2_H_DP: now also CN24.21
- net USB_HUB_EN: now also CN24.52
- net WIFI_CTRL: now also CN24.23
- net WIFI_EN: now also CN24.51
- net WOWLAN: now also CN24.11
- net USB1_DN: now reaches J4.103 (3)
- net USB1_DN: now also CN24.26
- net USB1_DP: now reaches J4.105 (5)
- net USB1_DP: now also CN24.35
- net USB1_TX1P_F: now reaches J4.152 (52)
- net USB1_TX1P_F: now also CN24.45
- net USB1_TX1N_F: now reaches J4.154 (54)
- net USB1_TX1N_F: now also CN24.16
- net USB1_RX1P: now reaches J4.158 (58)
- net USB1_RX1P: now also CN24.49
- net USB1_RX1N: now reaches J4.160 (60)
- net USB1_RX1N: now also CN24.12
- net DP_SS_RXN renamed USB1_RX2N
- net USB1_RX2N: now also CN24.13
- net DP_SS_RXP renamed USB1_RX2P
- net USB1_RX2P: now also CN24.48
- net DP_SS_TXN renamed USB1_TX2N_F
- net USB1_TX2N_F: now also CN24.17
- net DP_SS_TXP renamed USB1_TX2P_F
- net USB1_TX2P_F: now also CN24.44
- net TYPEC_AUXN renamed SBU2
- net SBU2: now also CN24.43
- net TYPEC_AUXP renamed SBU1
- net SBU1: now also CN24.18
- net USB1_DIR: no longer names the net of J4.38
- net USB1_MUX_EN: no longer names the net of J4.40
- net USBCC_INT_L renamed USBC1_INT_L
- net USBC1_INT_L: now also CN24.46
- new net FerriteGND_IO: CN24.61, CN24.62, CN24.63, CN24.64
- no-connect marks 98 -> 91

Commit message: update schematics and flex cable project
Parts:
- removed C111, C114, C115, C133, C134, C136, C139, C147, C21, C211, C215, C219, C59: 100nF, Capacitor_SMD:C_0603_1608Metric, symbol Device:C_Small
- removed C116, C131, C135, C137, C140: 10µF, Capacitor_SMD:C_0603_1608Metric, symbol Device:C_Small
- removed C117, C123, C19: 2.2µF, Capacitor_SMD:C_0603_1608Metric, symbol Device:C_Small
- removed C118, C120, C121, C124, C129, C130, C132, C138, C150, C155: 1µF, Capacitor_SMD:C_0603_1608Metric, symbol Device:C_Small
- removed C119, C122, C156: 100pF, Capacitor_SMD:C_0603_1608Metric, symbol Device:C_Small
- removed C125, C126, C127, C128: 1nF, Capacitor_SMD:C_0603_1608Metric, symbol Device:C_Small
- removed C213: 47µF, Capacitor_SMD:C_0805_2012Metric, symbol Device:C_Small
- removed C217: 4.7µF, Capacitor_SMD:C_0603_1608Metric, symbol Device:C_Small
- removed CN10, CN8: DF40C-40DP-0.4V, slate113:CONN-SMD_DF40C-40DP-0.4V, symbol slate113:DF40C-40DP-0.4V
- removed CN11: DF40C-30DP-0.4V, slate113:CONN-SMD_30P-P0.40_5001-BM0430-15-00, symbol slate113:DF40C-30DP-0.4V
- removed CN19: DF40C-24DP-0.4V, slate113:CONN-SMD_DF40C-24DP-0.4V, symbol slate113:DF40C-24DP-0.4V
- removed CN24: DF40C-60DP-0.4V, slate113:CONN-SMD_DF40C-60DP-0.4V, symbol slate113:DF40C-60DP-0.4V
- removed FB2: FerriteBead, Inductor_SMD:L_0603_1608Metric, symbol Device:FerriteBead
- removed FB6, FB7, FB8, FB9: 600Ω @ 100MHz, Inductor_SMD:L_0603_1608Metric, symbol Device:FerriteBead_Small
- removed FPC1: FPC0.5-24P, slate113:FPC-SMD_P0.50-24P_XJ-FGS, symbol slate113:FPC0.5-24P
- removed FPC2: FPC-0.5FX-6PWBH10, slate113:FPC-SMD_FPC-0.5FX-6PWBH10, symbol slate113:FPC-0.5FX-6PWBH10
- removed J4: DF40C-100DP-0.4V51*2, slate113:Raspberry-Pi-4-Compute-Module, symbol slate113:CM5_|_DF40C-100DP-0.4V51_*2
- removed LS1, LS2: Solder Pad, TestPoint:TestPoint_2Pads_Pitch2.54mm_Drill0.8mm, symbol Connector:Conn_01x02_Pin
- removed Q4: MMBT3904-C20526, slate113:SOT-23-3_L2.9-W1.3-P1.90-LS2.4-BR, symbol slate113:MMBT3904-C20526
- removed R100: 10kΩ, Resistor_SMD:R_0603_1608Metric, symbol Device:R
- removed R105, R17: 100kΩ, Resistor_SMD:R_0603_1608Metric, symbol Device:R_Small
- removed R106, R107: 560Ω, Resistor_SMD:R_0603_1608Metric, symbol Device:R_Small
- removed R108, R109, R122, R124, R126, R127, R128, R129, R74, R75, R96: 10kΩ, Resistor_SMD:R_0603_1608Metric, symbol Device:R_Small
- removed R67: 33Ω, Resistor_SMD:R_0603_1608Metric, symbol Device:R_Small
- removed R70: 10Ω, Resistor_SMD:R_0603_1608Metric, symbol Device:R_Small
- removed R71, R72, R73: 1kΩ, Resistor_SMD:R_0603_1608Metric, symbol Device:R_Small
- removed R97, R98: 4.7kΩ, Resistor_SMD:R_0603_1608Metric, symbol Device:R
- removed R99: 200kΩ, Resistor_SMD:R_0603_1608Metric, symbol Device:R_Small
- removed SW1, SW2: SW_Push, slate113:KEY-SMD_KMR2XXGXXX, symbol Switch:SW_Push
- removed U11: SiP32508DT, Package_TO_SOT_SMD:TSOT-23-6, symbol Power_Management:SiP32508DT
- removed U47: ES8388, slate113:QFN-28_L4.0-W4.0-P0.45-BL-EP, symbol slate113:ES8388
- removed U48, U49: TS5A23157DGSR, slate113:MSOP-10_L3.0-W3.0-P0.50-LS5.0-BL, symbol slate113:TS5A23157DGSR
- removed U50, U51: PAM8302AASCR, slate113:MSOP-8_L3.0-W3.0-P0.65-LS5.0-BL, symbol slate113:PAM8302AASCR
- removed U52: TPS7A0233PDBVR, slate113:SOT-23-5_L2.9-W1.6-P0.95-LS2.8-BR, symbol slate113:TPS7A0233PDBVR
- removed U62: PCA9306DCUR, slate113:SSOP-8_L2.0-W2.3-P0.50-LS3.1-BR, symbol slate113:PCA9306DCUR
- removed U63: AP2120N-2.8TRG1, slate113:SOT-23-3_L2.9-W1.3-P1.90-LS2.4-BR, symbol slate113:AP2120N-2.8TRG1
- removed U65: MSM381ADB001, slate113:MIC-SMD_5P_L3.5-W2.7-P0.82_MSM381ADB001, symbol slate113:MSM381ADB001
- removed U66: DF40B-10DS-0.4V, slate113:CONN-SMD_10P-P0.40_DF40B-10DS-0.4V-51, symbol slate113:DF40B-10DS-0.4V
- removed U67: SIP32508DT-T1-GE3, slate113:TSOT-23-6_L2.9-W1.6-P0.95-LS2.8-BR, symbol slate113:SIP32508DT-T1-GE3
- removed U68: SN74AHCT125PWR, slate113:TSSOP-14_L5.0-W4.4-P0.65-LS6.4-BL, symbol slate113:SN74AHCT125PWR
- removed U69: TCA9535PWR, slate113:TSSOP-24_L7.8-W4.4-P0.65-LS6.4-BL, symbol slate113:TCA9535PWR_C130204
- removed U8: ESD7104MUTAG_C2987068, slate113:DFN-10_L2.5-W1.0-P0.50-BL, symbol slate113:ESD7104MUTAG_C2987068
Connections:
- no-connect marks 91 -> 0
Other:
- added sheet Main Board Audio (MainBoard-Audio.kicad_sch)
- added sheet Main Board Display (MainBoard-Display.kicad_sch)
- added sheet Main Board Interfaces (MainBoard-Interfaces.kicad_sch)
- added sheet Main Board LED (MainBoard-LED.kicad_sch)
- added sheet Main Board Misc (MainBoard-Misc.kicad_sch)
- note removed: "1-100 CM5"
- note removed: "101-200 CM5"
- note removed: "2V8 LDO"
- note removed: "Audio LDO"
- note removed: "B2B > Carrier"
- note removed: "Buffer"
- note removed: "Carrier -> LED Status"
- note removed: "Controller"
- note removed: "Display Clamshell"
- note removed: "Ferrite"
- note removed: "GPIO Expander"
- note removed: "IO Connector"
- note removed: "Level Shifter"
- note removed: "M.2 Connector"
- note removed: "M.2 Power"
- note removed: "MOSFET"
- note removed: "Main > Radio"
- note removed: "PWR Declarations"
- note removed: "PWR Mezzanine"
- note removed: "PWR and RST BTNs"
- note removed: "Power Distributor"
- note removed: "Random Resistor"
- note removed: "Resistors"
- note removed: "Stereo Audio Codec Stuff"
- note removed: "TVS"
- note removed: "Touch Clamshell"
