File: Kicad Project/power.kicad_sch (KiCad schematic)
At the start: 47 parts, among them CN14 DF40C-30DP-0.4V, CN17 530480310, J2 TYPE-C16PIN, Q5 CSD17575Q3, Q6 CSD17575Q3, Q7 CSD17575Q3, Q8 CSD17575Q3, U2 CH224K, U3 BQ25792RQMR, U4 AP2112K-3.3TRG1, U5 AP2112K-1.8TRG1, U6 LP8556SQ-E09/NOPB, U9 TPS61088RHLR

Commit message: made some schematic changes to power
Parts:
- removed R10: 100kΩ, Resistor_SMD:R_0603_1608Metric, symbol Device:R
- added C251, C252, C253, C254, C41: GRM31CR71E106KA12L, slate113:C1206, symbol slate113:GRM31CR71E106KA12L
- added C255, C260, C264: 100nF, Capacitor_SMD:C_0603_1608Metric, symbol Device:C_Small
- added C256, C257, C261: 1.0µF, Capacitor_SMD:C_0603_1608Metric, symbol Device:C_Small
- added C258, C262, C263, C265: 10µF, Capacitor_SMD:C_0603_1608Metric, symbol Device:C_Small
- added C259: 0402B102K500NT, slate113:C0402, symbol slate113:0402B102K500NT
- added R10: 0402WGF5231TCE, slate113:R0402, symbol slate113:0402WGF5231TCE
- added R157: 0402WGF3012TCE, slate113:R0402, symbol slate113:0402WGF3012TCE
- added R158: 1kΩ, Resistor_SMD:R_0603_1608Metric, symbol Device:R_Small
- C157: value 4.7µF/10V/Ceramic -> 10µF; LCSC Part C77045 -> C380317; MPN GRM188R61C475KE11D -> TCC0603X5R106M160CT; Manufacturer Murata Electronics -> Samsung Electro-Mechanics
- R6: value 100kΩ -> 10kΩ; LCSC Part C25803 -> C840630; MPN 0603WAF1003T5E -> CR0603-FX-1002ELF; Manufacturer Yageo -> Bourns
Connections:
- net 1V8: now also C257.1
- net 3V3: now also U5.3 (EN), C256.1; no longer C8.1, L4.1, R7.1, U2.1 (VDD), U3.25 (SYS), U4.1 (VIN), U9.9 (VIN)
- net CM5_5V: now also C8.1, U4.1 (VIN), U4.3 (EN)
- net COMP: no longer C16.1
- net GND: now also R7.1, U2.3 (CFG3), U2.9 (CFG1), C251.2, C252.2, C253.2, C254.2, C255.1, C256.2, C257.2, C258.2, C259.2, C260.2, C261.1, C262.2, C263.2, C264.2, C265.2, C41.2, R157.1; no longer R16.2, R6.1
- net J2_VBUS: now also Q5.5 (D), R6.2, U3.9 (VAC1), R158.2; no longer U2.8 (VBUS)
- net REGN: now also R10.2; no longer C157.1
- net TS: now also R10.1, R157.2
- net VBAT: now also C265.1
- net VBUS: now also Q6.5 (D), Q8.5 (D), C262.1, C263.1, C264.1
- net VIN_EXT: no longer Q8.5 (D)
- net at U3.12 (~{QON}): no longer R6.2
- net SDRV: now reaches U3.24 (SDRV)
- net SDRV: now also C259.1
- net at C7.1, U3.29 (PMID): now also C157.1, C258.1, C260.1
- removed net VAC1: Q5.5 (D), Q6.5 (D), U2.2 (CFG2), U3.9 (VAC1)
- new net: C16.1, R16.2
- new net: C261.2, R158.1, U2.1 (VDD), U2.2 (CFG2)
- new net: R6.1, U2.8 (VBUS)
- new net VSYS: C251.1, C252.1, C253.1, C254.1, C255.2, C41.1, L4.1, U3.25 (SYS), U9.9 (VIN)
- no-connect marks 35 -> 31
Other:
- moved on the sheet: C16, C17, C6, C7, CN17, U2

Commit message: update schematics and flex cable project
Parts:
- removed C10: 10µF, Capacitor_SMD:C_0603_1608Metric, symbol Device:C_Small
- removed C11: 4.7µF, Capacitor_SMD:C_0603_1608Metric, symbol Device:C_Small
- removed C12: 2.2µF, Capacitor_SMD:C_0603_1608Metric, symbol Device:C_Small
- removed D1: B5819W, Diode_SMD:D_SOD-123, symbol Device:D
- removed L3: 10µH, slate113:IND-SMD_L7.1-W6.6, symbol Device:L
- removed R8: 205kΩ, Resistor_SMD:R_0603_1608Metric, symbol Device:R
- removed R9: 127kΩ, Resistor_SMD:R_0603_1608Metric, symbol Device:R
- removed U6: LP8556SQ-E09/NOPB, slate113:WQFN-24_L4.0-W4.0-P0.50-BL-EP2.5, symbol slate113:LP8556SQ-E09_NOPB
- added C269: 4.7µF, YX55069BCT2:C0805, symbol Device:C_Small
- added C271: 100 nF, YX55069BCT2:C_0603_1608Metric, symbol Device:C_Small
- added C272: 220 nF, YX55069BCT2:C0402, symbol YX55069BCT2:CL05B224KO5NNNC
- added C273: 10 uF, YX55069BCT2:C1206, symbol Device:C_Small
- added D53: S16, YX55069BCT2:SOD-123FL_L2.7-W1.8-LS3.8-RD, symbol YX55069BCT2:S16
- added L13: 10µH, slate113:IND-SMD_L7.1-W6.6, symbol Device:L
- added R166: 5 Ohm, YX55069BCT2:R0402, symbol YX55069BCT2:CSRT0402FT5R00
- added U16: TPS61165DBVR, YX55069BCT2:SOT-23-6_L2.9-W1.6-P0.95-LS2.8-BR, symbol YX55069BCT2:TPS61165DBVR
- C157, C258, C262, C263, C7: footprint Capacitor_SMD:C_0603_1608Metric -> Capacitor_SMD:C_1206_3216Metric; LCSC Part C380317 -> C77092; MPN TCC0603X5R106M160CT -> GRM31CR61H106KA12L; Manufacturer Samsung Electro-Mechanics -> Murata
- R158: footprint Resistor_SMD:R_0603_1608Metric -> Resistor_SMD:R_1206_3216Metric; LCSC Part C118155 -> C4279633; MPN ERJ3EKF1001V -> AC1206FR-7W1KL; Manufacturer Panasonic -> YAGEO
Connections:
- net CM5_5V: now also C269.2, C271.1, L13.1, U16.1 (VIN)
- net GND: now also C269.1, C271.2, C272.1, C273.2, R166.2, U16.4 (GND)
- net L1P1: now also D53.2 (A), L13.2, U16.3 (SW)
- net LCD_LED_K: now also R166.1, U16.6 (FB)
- net LCD_PWM: now also U16.2 (CTRL)
- net LCD_LED_A: now reaches CN14.22
- net LCD_LED_A: now also C273.1, D53.1 (C)
- net at U2.4 (DP): now also U2.5 (DM)
- new net: C272.2, U16.5 (COMP)
- no-connect marks 31 -> 23
Other:
- note added: "Backlight LED Driver"
