File: Kicad Project/powerflex.kicad_sch (KiCad schematic)
At the start: 2 parts, among them CN3 DF40C-30DS-0.4V, CN7 DF40C-30DS-0.4V

Commit message: update schematics and flex cable project
Parts:
- removed CN3: DF40C-30DS-0.4V, slate113:CONN-SMD_DF40C-30DS-0.4V51, symbol slate113:DF40C-30DS-0.4V
- added CN?: DF40C-30DS-0.4V, slate113:CONN-SMD_DF40C-30DS-0.4V51, symbol slate113:DF40C-30DS-0.4V
Connections:
- net 1V8: now also CN?.5
- net 3V3: now also CN?.4
- net BQ_INT: now also CN?.7
- net CM5_5V: now also CN?.2, CN?.3
- net GND: now also CN?.1, CN?.11, CN?.12, CN?.6
- net I2C0_SCL: now also CN?.8
- net I2C0_SDA: now also CN?.9
- net LCD_LED_K: now also CN?.21
- net LCD_PWM: now also CN?.19
- net VBOOST: now also CN?.20
- net VBUS: now also CN?.13, CN?.14, CN?.15
- net VIN_EXT: now also CN?.16, CN?.17, CN?.18
- net LCD_LED_A: now reaches CN7.22
- net LCD_LED_A: now also CN?.22
- no-connect marks 20 -> 18
