File: Kicad Project/slate113.kicad_sch (KiCad schematic)
At the start: 0 parts

Commit message: made some schematic changes to power
Parts:
- added BT1: MY-1220-03, slate113:BAT-SMD_MY-1220-03, symbol slate113:MY-1220-03
- added C30, C31: 100nF, Capacitor_SMD:C_0603_1608Metric, symbol Device:C_Small
- added CN1: DF40C-10DP-0.4V, slate113:CONN-SMD_10P-P0.40_DF40C-10DP-0.4V-51, symbol slate113:DF40C-10DP-0.4V
- added D53: TPD4E05U06DQAR, slate113:USON-10_L2.5-W1.0-P0.50-BL, symbol slate113:TPD4E05U06DQAR_C138714
- added R111, R121, R123, R156: 10kΩ, Resistor_SMD:R_0603_1608Metric, symbol Device:R_Small
- added R125, R154, R155, R34, R35: 100kΩ, Resistor_SMD:R_0603_1608Metric, symbol Device:R_Small
- added U7: SN74LVC1G08DBVR, slate113:SOT-23-5_L3.0-W1.7-P0.95-LS2.8-BR, symbol slate113:SN74LVC1G08DBVR

Commit message: update schematics and flex cable project
Parts:
- removed BT1: MY-1220-03, slate113:BAT-SMD_MY-1220-03, symbol slate113:MY-1220-03
- removed C30, C31: 100nF, Capacitor_SMD:C_0603_1608Metric, symbol Device:C_Small
- removed CN1: DF40C-10DP-0.4V, slate113:CONN-SMD_10P-P0.40_DF40C-10DP-0.4V-51, symbol slate113:DF40C-10DP-0.4V
- removed D53: TPD4E05U06DQAR, slate113:USON-10_L2.5-W1.0-P0.50-BL, symbol slate113:TPD4E05U06DQAR_C138714
- removed R111, R121, R123, R156: 10kΩ, Resistor_SMD:R_0603_1608Metric, symbol Device:R_Small
- removed R125, R154, R155, R34, R35: 100kΩ, Resistor_SMD:R_0603_1608Metric, symbol Device:R_Small
- removed U7: SN74LVC1G08DBVR, slate113:SOT-23-5_L3.0-W1.7-P0.95-LS2.8-BR, symbol slate113:SN74LVC1G08DBVR
