File: Flex Cables Kicad Project/Flex Cables Kicad Project.kicad_sch (KiCad schematic)
At the start: 0 parts

Commit message: update schematics and flex cable project
Other:
- added sheet IO Flex (IOFlex.kicad_sch)
- added sheet LED Bar (LEDBar.kicad_sch)
- added sheet M.2 Flex (M.2Flex.kicad_sch)
- added sheet Power Flex (PowerFlex.kicad_sch)
- added sheet Radio Flex (RadioFlex.kicad_sch)
- added sheet Side Buttons Flex (SideButtonsFlex.kicad_sch)
- added sheet Slate Connect Flex (SlateConnectFlex.kicad_sch)
