File: Flex Cables Kicad Project/Flex Cables Kicad Project.kicad_pcb (KiCad board)
At the start: 2 copper layers, 10.1 x 70.9 mm, 105 parts, among them CN1 DF40C-30DS-0.4V, CN15 DF40C-24DS-0.4V, CN16 DF40C-24DS-0.4V, CN18 DF40C-10DP-0.4V, CN2 DF40C-60DS-0.4V, CN3 DF40C-60DS-0.4V, CN4 DF40C-40DS-0.4V, CN6 DF40C-40DS-0.4V, CN7 DF40C-30DS-0.4V, SW1 B3U-1000P, SW2 B3U-1000P, SW3 B3U-1000P, SW4 B3U-1000P, U1 DF40C-10DS-0.4V

Commit message: worked on more flexes
Parts:
- added CN5: DF40C-40DS-0.4V, slate113:CONN-SMD_DF40C-40DS-0.4V51, F.Cu at (153.2, 44.2)
- added CN8: DF40C-40DS-0.4V, slate113:CONN-SMD_DF40C-40DS-0.4V51, F.Cu at (153.2, 94.2)
- moved CN16 123.2 mm to (184.8, 109.2)
- moved CN15 96.4 mm to (184.8, 44.2)
- moved CN6 94.1 mm to (169.4, 85.5), turned to 180 degrees
- moved CN4 93.2 mm to (169.4, 45.5)
Routing:
- net GND: track 265.2 -> 789.5 mm, vias 4 -> 14
- net VIN_EXT: track 206.4 -> 363.3 mm, vias 4 -> 8
- net VBUS: track 193.3 -> 348.7 mm
- net RP_ACC_AUX0: track 0.00 -> 118.4 mm, vias 0 -> 2
- net RP_ACC_IRQ0: track 0.00 -> 116.7 mm, vias 0 -> 2
- net RP_ACC_MISO: track 0.00 -> 115.7 mm, vias 0 -> 2
- net 3V3: track 67.5 -> 152.8 mm
- net LED_PWR_EN: track 0.00 -> 62.4 mm
- net LED_DATA_3V3: track 0.00 -> 62.4 mm
- net CM5_UART_TX: track 0.00 -> 62.4 mm
- net CM5_ACC_AUX0: track 0.00 -> 59.2 mm, vias 0 -> 2
- net CM5_ACC_MISO: track 0.00 -> 58.0 mm, vias 0 -> 2
- net CM5_ACC_IRQ0: track 0.00 -> 56.4 mm, vias 0 -> 2
- net CM5_ACC_SCK: track 0.00 -> 55.3 mm, vias 0 -> 2
- net RP_ACC_SCK: track 0.00 -> 53.9 mm, vias 0 -> 2
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Other:
- board size 10.1 x 70.9 mm -> 41.6 x 72 mm
