File: Flex Cables Kicad Project/SlateConnectFlex.kicad_sch (KiCad schematic)
At the start: 0 parts

Commit message: worked on more flexes
Parts:
- added CN5, CN8: DF40C-40DS-0.4V, slate113:CONN-SMD_DF40C-40DS-0.4V51, symbol slate113:DF40C-40DS-0.4V
Connections:
- new net 3V3: CN5.11, CN8.11
- new net CM5_ACC_AUX0: CN5.28, CN8.28
- new net CM5_ACC_AUX1: CN5.29, CN8.29
- new net CM5_ACC_CS0_N: CN5.25, CN8.25
- new net CM5_ACC_IRQ0: CN5.26, CN8.26
- new net CM5_ACC_MISO: CN5.24, CN8.24
- new net CM5_ACC_MOSI: CN5.23, CN8.23
- new net CM5_ACC_RESET_N: CN5.27, CN8.27
- new net CM5_ACC_SCK: CN5.22, CN8.22
- new net GND: CN5.1, CN5.2, CN5.3, CN5.4, CN8.1, CN8.2, CN8.3, CN8.4
- new net RP_ACC_AUX0: CN5.36, CN8.36
- new net RP_ACC_AUX1: CN5.37, CN8.37
- new net RP_ACC_CS0_N: CN5.33, CN8.33
- new net RP_ACC_IRQ0: CN5.34, CN8.34
- new net RP_ACC_MISO: CN5.32, CN8.32
- new net RP_ACC_MOSI: CN5.31, CN8.31
- new net RP_ACC_RESET_N: CN5.35, CN8.35
- new net RP_ACC_SCK: CN5.30, CN8.30
- new net SC_ID_SCL: CN5.13, CN8.13
- new net SC_ID_SDA: CN5.12, CN8.12
- new net VBUS: CN5.5, CN5.6, CN5.7, CN8.5, CN8.6, CN8.7
- new net VIN_EXT: CN5.10, CN5.8, CN5.9, CN8.10, CN8.8, CN8.9
- no-connect marks 0 -> 22
